File: demos/pic_programmer/pic_programmer.sch (KiCad schematic (older format))
At the start: 56 parts, among them J1 DB9-FEMAL, P1 CONN_2, P101 CONN_1, P102 CONN_1, P103 CONN_1, P104 CONN_1, P105 CONN_1, P106 CONN_1, Q1 BC237, Q2 BC307, Q3 BC307, U2 74HC125, U3 7805, U4 LT1373

Commit message: New upstream version 5.0.0~rc3+dfsg1
Parts:
- P101, P102, P103, P104, P105, P106: symbol pic_programmer_schlib:CONN_1 -> pic_programmer_schlib:MOUNTING_HOLE
Connections:
- no-connect marks 12 -> 6
Changed lines of the file:
@@
 $EndComp
 $Comp
-L pic_programmer_schlib:CONN_1 P101
+L pic_programmer_schlib:MOUNTING_HOLE P101
 U 1 1 54020BEA
 P 6400 6800
@@
 $EndComp
 $Comp
-L pic_programmer_schlib:CONN_1 P102
+L pic_programmer_schlib:MOUNTING_HOLE P102
 U 1 1 54020DA9
 P 6400 6950
@@
 $EndComp
 $Comp
-L pic_programmer_schlib:CONN_1 P103
+L pic_programmer_schlib:MOUNTING_HOLE P103
 U 1 1 54020DC2
 P 6400 7100
@@
 $EndComp
 $Comp
-L pic_programmer_schlib:CONN_1 P104
+L pic_programmer_schlib:MOUNTING_HOLE P104
 U 1 1 54020DE3
 P 6400 7250
@@
 $EndComp
 $Comp
-L pic_programmer_schlib:CONN_1 P105
+L pic_programmer_schlib:MOUNTING_HOLE P105
 U 1 1 54020E5D
 P 6400 7400
@@
 $EndComp
 $Comp
-L pic_programmer_schlib:CONN_1 P106
+L pic_programmer_schlib:MOUNTING_HOLE P106
 U 1 1 54020E76
 P 6400 7550
@@
 Text Notes 6050 7700 0    40   Italic 0
 Mounting holes
-NoConn ~ 6250 6800
-NoConn ~ 6250 6950
-NoConn ~ 6250 7100
-NoConn ~ 6250 7250
-NoConn ~ 6250 7400
-NoConn ~ 6250 7550
 Wire Wire Line
 	3850 2700 3850 2750
