File: demos/pic_programmer/pic_sockets.sch (KiCad schematic (older format))
At the start: 7 parts, among them P2 SUPP28, P3 SUPP40, U1 24Cxx, U5 PIC_18_PINS, U6 PIC_8_PINS

Commit message: Imported Upstream version 0.0.20070525
Parts:
- added C8: 100nF, symbol C
Connections:
- net labels added: VCC_PIC
- wire segments 27 -> 28
Changed lines of the file:
@@
 EESchema Schematic File Version 1
-LIBS:power,device,conn,linear,regul,74xx,cmos4000,adc-dac,memory,xilinx,special,microcontrollers,microchip,analog_switches,motorola,intel,audio,interface,digital-audio,philips,display,cypress,siliconi,contrib,.\pic_programmer.cache
+LIBS:power,device,conn,linear,regul,74xx,cmos4000,adc-dac,memory,xilinx,special,microcontrollers,dsp,microchip,analog_switches,motorola,texas,intel,audio,interface,digital-audio,philips,display,cypress,siliconi,contrib,valves,.\pic_programmer.cache
 EELAYER 23  0
 EELAYER END
 $Descr A4 11700 8267
 Sheet 2 2
-Title "Pic programmer: Pic sockets"
-Date "16 may 2006"
-Rev "1"
+Title "JDM - COM84 PIC Programmer with 13V DC/DC converter"
+Date "16 may 2007"
+Rev "3"
 Comp "KiCad"
 Comment1 ""
@@
 Comment4 ""
 $EndDescr
-$Comp
-L GND #PWR33
+Wire Wire Line
+	3700 7000 3700 6900
+Wire Wire Line
+	2350 2150 3100 2150
+Wire Wire Line
+	10250 1800 9400 1800
+Wire Wire Line
+	9400 1700 10200 1700
+Wire Wire Line
+	8200 1700 7450 1700
+Connection ~ 2950 1100
+Wire Wire Line
+	2950 1100 3150 1100
+Connection ~ 2950 1200
+Wire Wire Line
+	2950 1250 2950 1000
+Wire Wire Line
+	2950 1000 3150 1000
+Wire Wire Line
+	3150 1200 2950 1200
+Wire Wire Line
+	4550 1400 5350 1400
+Wire Wire Line
+	5400 1300 4550 1300
+Wire Wire Line
+	10500 4250 9650 4250
+Wire Wire Line
+	9650 4150 10450 4150
+Wire Wire Line
+	8450 4150 7700 4150
+Wire Wire Line
+	2500 4850 2300 4850
+Wire Wire Line
+	4900 5150 4050 5150
+Wire Wire Line
+	4050 5000 4850 5000
+Wire Wire Line
+	2500 4700 1750 4700
+Wire Wire Line
+	5400 2850 4550 2850
+Wire Wire Line
+	4550 2450 5350 2450
+Wire Wire Line
+	3100 3150 2350 3150
+Wire Wire Line
+	2300 4850 2300 4900
+Wire Wire Line
+	4850 4850 4050 4850
+Wire Wire Line
+	10200 2500 9400 2500
+Wire Wire Line
+	10450 4950 9650 4950
+Wire Wire Line
+	8450 5150 7650 5150
+Wire Wire Line
+	3700 6900 4550 6900
+Wire Wire Line
+	4550 6900 4550 7000
+Text Label 3950 6900 0    60   ~
+VCC_PIC
+$Comp
+L GND #PWR036
+U 1 1 4639BE2E
+P 4550 7400
+F 0 "#PWR036" H 4550 7400 30  0001 C C
+F 1 "GND" H 4550 7330 30  0001 C C
+	1    4550 7400
+	1    0    0    -1
+$EndComp
+$Comp
+L C C8
+U 1 1 4639BE2C
+P 4550 7200
+F 0 "C8" H 4600 7300 50  0000 L C
+F 1 "100nF" H 4600 7100 50  0000 L C
+	1    4550 7200
+	1    0    0    -1
+$EndComp
+Text GLabel 2350 2150 0    60   Input
+VCC_PIC
+Text Label 2550 2150 0    60   ~
+VCC_PIC
+Text Label 7650 5150 0    60   ~
+VCC_PIC
+Text Label 9900 4950 0    60   ~
+VCC_PIC
+Text Label 9650 2500 0    60   ~
+VCC_PIC
+$Comp
+L GND #PWR037
+U 1 1 442A8794
+P 8450 5250
+F 0 "#PWR037" H 8450 5250 30  0001 C C
+F 1 "GND" H 8450 5180 30  0001 C C
+	1    8450 5250
+	0    1    1    0
+$EndComp
+Text Label 4300 4850 0    60   ~
+VCC_PIC
+$Comp
+L GND #PWR038
 U 1 1 443CCA5D
 P 8450 4850
-F 0 "#PWR33" H 8450 4850 30  0001 C C
+F 0 "#PWR038" H 8450 4850 30  0001 C C
 F 1 "GND" H 8450 4780 30  0001 C C
 	1    8450 4850
@@
 NoConn ~ 8200 1900
 NoConn ~ 8200 1800
-Wire Wire Line
-	9400 2500 9450 2500
-$Comp
-L VCC #PWR46
-U 1 1 443697F0
-P 9450 2500
-F 0 "#PWR46" H 9450 2600 30  0001 C C
-F 1 "VCC" H 9450 2600 30  0000 C C
-	1    9450 2500
-	0    1    1    0
-$EndComp
-$Comp
-L GND #PWR32
+$Comp
+L GND #PWR039
 U 1 1 443697C7
 P 9400 2600
-F 0 "#PWR32" H 9400 2600 30  0001 C C
+F 0 "#PWR039" H 9400 2600 30  0001 C C
 F 1 "GND" H 9400 2530 30  0001 C C
 	1    9400 2600
@@
 $EndComp
 $Comp
-L GND #PWR31
+L GND #PWR040
 U 1 1 443697C3
 P 8200 2400
-F 0 "#PWR31" H 8200 2400 30  0001 C C
+F 0 "#PWR040" H 8200 2400 30  0001 C C
 F 1 "GND" H 8200 2330 30  0001 C C
 	1    8200 2400
 	0    1    1    0
 $EndComp
-Wire Wire Line
-	10250 1800 9400 1800
-Wire Wire Line
-	9400 1700 10200 1700
 Text Label 9550 1800 0    60   ~
 CLOCK-RB6
 Text Label 9550 1700 0    60   ~
 DATA-RB7
-Wire Wire Line
-	8200 1700 7450 1700
 Text Label 7550 1700 0    60   ~
 VPP-MCLR
@@
 $EndComp
 $Comp
-L GND #PWR30
+L GND #PWR041
 U 1 1 442AA147
 P 3700 7400
-F 0 "#PWR30" H 3700 7400 30  0001 C C
+F 0 "#PWR041" H 3700 7400 30  0001 C C
 F 1 "GND" H 3700 7330 30  0001 C C
 	1    3700 7400
-	1    0    0    -1
-$EndComp
-$Comp
-L VCC #PWR45
-U 1 1 442AA146
-P 3700 7000
-F 0 "#PWR45" H 3700 7100 30  0001 C C
-F 1 "VCC" H 3700 7100 30  0000 C C
-	1    3700 7000
 	1    0    0    -1
 $EndComp
@@
 $EndComp
 $Comp
-L GND #PWR29
+L GND #PWR042
 U 1 1 442AA138
 P 2700 7400
-F 0 "#PWR29" H 2700 7400 30  0001 C C
+F 0 "#PWR042" H 2700 7400 30  0001 C C
 F 1 "GND" H 2700 7330 30  0001 C C
 	1    2700 7400
@@
 $EndComp
 $Comp
-L VCC #PWR44
+L VCC #PWR043
 U 1 1 442AA134
 P 2700 7000
-F 0 "#PWR44" H 2700 7100 30  0001 C C
+F 0 "#PWR043" H 2700 7100 30  0001 C C
 F 1 "VCC" H 2700 7100 30  0000 C C
 	1    2700 7000
@@
 NoConn ~ 8450 4350
 NoConn ~ 8450 4250
-Wire Wire Line
-	9650 4950 9700 4950
-$Comp
-L VCC #PWR43
-U 1 1 442A896B
-P 9700 4950
-F 0 "#PWR43" H 9700 5050 30  0001 C C
-F 1 "VCC" H 9700 5050 30  0000 C C
-	1    9700 4950
-	0    1    1    0
-$EndComp
-$Comp
-L GND #PWR28
+$Comp
+L GND #PWR044
 U 1 1 442A896A
 P 9650 5050
-F 0 "#PWR28" H 9650 5050 30  0001 C C
+F 0 "#PWR044" H 9650 5050 30  0001 C C
 F 1 "GND" H 9650 4980 30  0001 C C
 	1    9650 5050
@@
 $EndComp
 NoConn ~ 4550 1100
-Connection ~ 2950 1100
-Wire Wire Line
-	3150 1100 2950 1100
-Connection ~ 2950 1200
-Wire Wire Line
-	2950 1250 2950 1000
-Wire Wire Line
-	2950 1000 3150 1000
-Wire Wire Line
-	3150 1200 2950 1200
-$Comp
-L GND #PWR27
+$Comp
+L GND #PWR045
 U 1 1 442A8838
 P 2950 1250
-F 0 "#PWR27" H 2950 1250 30  0001 C C
+F 0 "#PWR045" H 2950 1250 30  0001 C C
 F 1 "GND" H 2950 1180 30  0001 C C
 	1    2950 1250
 	1    0    0    -1
 $EndComp
-Wire Wire Line
-	4550 1400 5350 1400
 Text Label 4700 1400 0    60   ~
 DATA-RB7
-Wire Wire Line
-	5400 1300 4550 1300
 Text Label 4700 1300 0    60   ~
 CLOCK-RB6
@@
 	1    0    0    -1
 $EndComp
-Wire Wire Line
-	10500 4250 9650 4250
-Wire Wire Line
-	9650 4150 10450 4150
 Text Label 9800 4250 0    60   ~
 CLOCK-RB6
 Text Label 9800 4150 0    60   ~
 DATA-RB7
-Wire Wire Line
-	8450 4150 7700 4150
 Text Label 7800 4150 0    60   ~
 VPP-MCLR
-Wire Wire Line
-	8400 5150 8450 5150
-$Comp
-L VCC #PWR42
-U 1 1 442A8796
-P 8400 5150
-F 0 "#PWR42" H 8400 5250 30  0001 C C
-F 1 "VCC" H 8400 5250 30  0000 C C
-	1    8400 5150
-	0    -1   -1   0
-$EndComp
-$Comp
-L GND #PWR26
-U 1 1 442A8794
-P 8450 5250
-F 0 "#PWR26" H 8450 5250 30  0001 C C
-F 1 "GND" H 8450 5180 30  0001 C C
-	1    8450 5250
-	0    1    1    0
-$EndComp
 NoConn ~ 2500 4400
 NoConn ~ 4050 5450
@@
 	1    0    0    -1
 $EndComp
-Wire Wire Line
-	2500 4850 2300 4850
-Wire Wire Line
-	4050 4850 4200 4850
 NoConn ~ 4550 3150
 NoConn ~ 3100 2850
 NoConn ~ 3100 2450
-Wire Wire Line
-	4900 5150 4050 5150
-Wire Wire Line
-	4050 5000 4850 5000
 Text Label 4200 5150 0    60   ~
 CLOCK-RB6
 Text Label 4200 5000 0    60   ~
 DATA-RB7
-Wire Wire Line
-	2500 4700 1750 4700
 Text Label 1850 4700 0    60   ~
 VPP-MCLR
-Wire Wire Line
-	5400 2850 4550 2850
-Wire Wire Line
-	4550 2450 5350 2450
-Wire Wire Line
-	3100 3150 2350 3150
 Text Label 2450 3150 0    60   ~
 VPP-MCLR
@@
 Text GLabel 1350 4050 0    60   Input
 DATA-RB7
-Wire Wire Line
-	2300 4850 2300 4900
-Wire Wire Line
-	4200 4850 4200 4800
-Wire Wire Line
-	3100 2150 3050 2150
-Wire Wire Line
-	3050 2150 3050 2050
-$Comp
-L GND #PWR25
+$Comp
+L GND #PWR046
 U 1 1 442A820F
 P 2300 4900
-F 0 "#PWR25" H 2300 4900 30  0001 C C
+F 0 "#PWR046" H 2300 4900 30  0001 C C
 F 1 "GND" H 2300 4830 30  0001 C C
 	1    2300 4900
@@
 $EndComp
 $Comp
-L GND #PWR24
+L GND #PWR047
 U 1 1 442A8205
 P 4550 2150
-F 0 "#PWR24" H 4550 2150 30  0001 C C
+F 0 "#PWR047" H 4550 2150 30  0001 C C
 F 1 "GND" H 4550 2080 30  0001 C C
 	1    4550 2150
@@
 $EndComp
 $Comp
-L VCC #PWR41
-U 1 1 442A81FE
-P 3050 2050
-F 0 "#PWR41" H 3050 2150 30  0001 C C
-F 1 "VCC" H 3050 2150 30  0000 C C
-	1    3050 2050
-	1    0    0    -1
-$EndComp
-$Comp
-L VCC #PWR40
-U 1 1 442A81F9
-P 4200 4800
-F 0 "#PWR40" H 4200 4900 30  0001 C C
-F 1 "VCC" H 4200 4900 30  0000 C C
-	1    4200 4800
-	1    0    0    -1
-$EndComp
-$Comp
