File: demos/pic_programmer/pic_sockets.sch (KiCad schematic (older format))
At the start: 8 parts, among them P2 SUPP28, P3 SUPP40, U1 24Cxx, U5 PIC_18_PINS, U6 PIC_8_PINS

Commit message: Imported Upstream version 4.0.0~rc1
Parts:
- removed C8: 100nF, symbol C
- C6, C7: footprint (none) -> discret:C1-1
- P2: footprint (none) -> dip_sockets:DIP-28__300_ELL
- P3: footprint (none) -> sockets:40tex-Ell600
- U1, U6: footprint (none) -> dip_sockets:DIP-8__300_ELL
- U5: footprint (none) -> dip_sockets:DIP-18__300_ELL
Connections:
- net labels removed: VCC
- wire segments 28 -> 46

Commit message: New upstream version 5.0.0~rc1+dfsg1
Parts:
- C6, C7: footprint discret:C1-1 -> Capacitor_THT:C_Disc_D5.1mm_W3.2mm_P5.00mm; symbol C -> pic_programmer_schlib:C
- P2: footprint dip_sockets:DIP-28__300_ELL -> Package_DIP:DIP-28_W7.62mm_Socket_LongPads; symbol SUPP28 -> pic_programmer_schlib:SUPP28
- P3: symbol SUPP40 -> pic_programmer_schlib:SUPP40
- U1: footprint dip_sockets:DIP-8__300_ELL -> Package_DIP:DIP-8_W7.62mm_Socket_LongPads; symbol 24C16 -> pic_programmer_schlib:24C16
- U5: footprint dip_sockets:DIP-18__300_ELL -> Package_DIP:DIP-18_W7.62mm_Socket_LongPads; symbol PIC16F54 -> pic_programmer_schlib:PIC16F54
- U6: footprint dip_sockets:DIP-8__300_ELL -> Package_DIP:DIP-8_W7.62mm_Socket_LongPads; symbol PIC12C508A -> pic_programmer_schlib:PIC12C508A
Connections:
- wire segments 46 -> 66
Changed lines of the file:
@@
-EESchema Schematic File Version 2
-LIBS:pic_programmer_schlib
-LIBS:power
+EESchema Schematic File Version 4
 LIBS:pic_programmer-cache
-EELAYER 25 0
+EELAYER 26 0
 EELAYER END
 $Descr A4 11693 8268
@@
 Connection ~ 2800 1300
 Wire Wire Line
-	2800 1100 2800 1350
+	2800 1100 2800 1200
 Wire Wire Line
 	2800 1100 3000 1100
@@
 	3000 1300 2800 1300
 Wire Wire Line
-	4400 1500 10000 1500
-Wire Wire Line
-	4400 1400 10100 1400
+	4400 1500 5300 1500
+Wire Wire Line
+	4400 1400 5400 1400
 Wire Wire Line
 	10100 4000 9200 4000
@@
 VCC_PIC
 $Comp
-L GND #PWR036
+L pic_programmer_schlib:GND #PWR036
 U 1 1 442A8794
 P 8000 5000
@@
 VCC_PIC
 $Comp
-L GND #PWR037
+L pic_programmer_schlib:GND #PWR037
 U 1 1 443CCA5D
 P 8000 4600
@@
 NoConn ~ 8000 2000
 $Comp
-L GND #PWR038
+L pic_programmer_schlib:GND #PWR038
 U 1 1 443697C7
 P 9200 2800
@@
 $EndComp
 $Comp
-L GND #PWR039
+L pic_programmer_schlib:GND #PWR039
 U 1 1 443697C3
 P 8000 2600
@@
 VPP-MCLR
 $Comp
-L SUPP28 P2
+L pic_programmer_schlib:SUPP28 P2
 U 1 1 4436967E
 P 8600 2550
 F 0 "P2" H 8600 3350 70  0000 C CNN
 F 1 "SUPP28" H 8600 1700 70  0000 C CNN
-F 2 "dip_sockets:DIP-28__300_ELL" H 8600 1600 60  0000 C CNN
+F 2 "Package_DIP:DIP-28_W7.62mm_Socket_LongPads" H 8600 1600 15  0000 C CNN
 F 3 "" H 8600 2550 60  0001 C CNN
 	1    8600 2550
@@
 $EndComp
 $Comp
-L GND #PWR040
+L pic_programmer_schlib:GND #PWR040
 U 1 1 442AA147
-P 3300 7050
-F 0 "#PWR040" H 3300 7050 30  0001 C CNN
-F 1 "GND" H 3300 6980 30  0001 C CNN
-F 2 "" H 3300 7050 60  0001 C CNN
-F 3 "" H 3300 7050 60  0001 C CNN
-	1    3300 7050
-	1    0    0    -1
-$EndComp
-$Comp
-L C C7
+P 3300 6950
+F 0 "#PWR040" H 3300 6950 30  0001 C CNN
+F 1 "GND" H 3300 6880 30  0001 C CNN
+F 2 "" H 3300 6950 60  0001 C CNN
+F 3 "" H 3300 6950 60  0001 C CNN
+	1    3300 6950
+	1    0    0    -1
+$EndComp
+$Comp
+L pic_programmer_schlib:C C7
 U 1 1 442AA145
-P 3300 6800
-F 0 "C7" H 3350 6900 50  0000 L CNN
-F 1 "100nF" H 3350 6700 50  0000 L CNN
-F 2 "discret:C1-1" H 3650 6600 60  0000 C CNN
-F 3 "" H 3300 6800 60  0001 C CNN
-	1    3300 6800
-	1    0    0    -1
-$EndComp
-$Comp
-L GND #PWR041
+P 3300 6750
+F 0 "C7" H 3350 6850 50  0000 L CNN
+F 1 "100nF" H 3350 6650 50  0000 L CNN
+F 2 "Capacitor_THT:C_Disc_D5.1mm_W3.2mm_P5.00mm" H 3500 6600 10  0000 C CNN
+F 3 "" H 3300 6750 60  0001 C CNN
+	1    3300 6750
+	1    0    0    -1
+$EndComp
+$Comp
+L pic_programmer_schlib:GND #PWR041
 U 1 1 442AA138
-P 2400 7050
-F 0 "#PWR041" H 2400 7050 30  0001 C CNN
-F 1 "GND" H 2400 6980 30  0001 C CNN
-F 2 "" H 2400 7050 60  0001 C CNN
-F 3 "" H 2400 7050 60  0001 C CNN
-	1    2400 7050
+P 2400 6950
+F 0 "#PWR041" H 2400 6950 30  0001 C CNN
+F 1 "GND" H 2400 6880 30  0001 C CNN
+F 2 "" H 2400 6950 60  0001 C CNN
+F 3 "" H 2400 6950 60  0001 C CNN
+	1    2400 6950
 	1    0    0    -1
 $EndComp
@@
 NoConn ~ 8000 4000
 $Comp
-L GND #PWR042
+L pic_programmer_schlib:GND #PWR042
 U 1 1 442A896A
 P 9200 4800
@@
 $EndComp
 $Comp
-L SUPP40 P3
+L pic_programmer_schlib:SUPP40 P3
 U 1 1 442A88ED
 P 8600 4850
 F 0 "P3" H 8600 5950 70  0000 C CNN
 F 1 "SUPP40" H 8600 3700 70  0000 C CNN
-F 2 "sockets:40tex-Ell600" H 8600 3600 60  0000 C CNN
+F 2 "sockets:40tex-Ell600" H 8600 3600 15  0000 C CNN
 F 3 "" H 8600 4850 60  0001 C CNN
 	1    8600 4850
@@
 NoConn ~ 4400 1200
 $Comp
-L GND #PWR043
+L pic_programmer_schlib:GND #PWR043
 U 1 1 442A8838
 P 2800 1350
@@
 CLOCK-RB6
 $Comp
-L 24C16 U1
+L pic_programmer_schlib:24C16 U1
 U 1 1 442A87F7
 P 3700 1300
 F 0 "U1" H 3850 1650 60  0000 C CNN
 F 1 "24Cxx" H 3900 950 60  0000 C CNN
-F 2 "dip_sockets:DIP-8__300_ELL" H 4450 850 60  0000 C CNN
+F 2 "Package_DIP:DIP-8_W7.62mm_Socket_LongPads" H 3900 900 10  0000 C CNN
 F 3 "" H 3700 1300 60  0001 C CNN
 	1    3700 1300
@@
 NoConn ~ 2950 4000
 $Comp
-L PIC16F54 U5
+L pic_programmer_schlib:PIC16F54 U5
 U 1 1 442A81A7
 P 3750 4600
 F 0 "U5" H 3750 5350 60  0000 C CNN
 F 1 "PIC_18_PINS" H 3750 3800 60  0000 C CNN
-F 2 "dip_sockets:DIP-18__300_ELL" H 3800 3700 60  0000 C CNN
+F 2 "Package_DIP:DIP-18_W7.62mm_Socket_LongPads" H 3800 3700 15  0000 C CNN
 F 3 "" H 3750 4600 60  0001 C CNN
 	1    3750 4600
@@
 DATA-RB7
 $Comp
-L GND #PWR044
+L pic_programmer_schlib:GND #PWR044
 U 1 1 442A820F
 P 2750 4650
@@
 $EndComp
 $Comp
-L GND #PWR045
+L pic_programmer_schlib:GND #PWR045
 U 1 1 442A8205
 P 4450 2400
@@
 $EndComp
 $Comp
-L PIC12C508A U6
+L pic_programmer_schlib:PIC12C508A U6
 U 1 1 442A81A5
 P 3750 2900
 F 0 "U6" H 3700 3600 60  0000 C CNN
-F 1 "PIC_8_PINS" H 3750 2200 60  0000 C CNN
-F 2 "dip_sockets:DIP-8__300_ELL" H 3750 2100 60  0000 C CNN
+F 1 "PIC_8_PINS" H 3750 2250 60  0000 C CNN
+F 2 "Package_DIP:DIP-8_W7.62mm_Socket_LongPads" H 3750 2150 15  0000 C CNN
 F 3 "" H 3750 2900 60  0001 C CNN
 	1    3750 2900
@@
 $EndComp
 $Comp
-L GND #PWR046
+L pic_programmer_schlib:GND #PWR046
 U 1 1 52C92629
 P 3700 1850
@@
 VCC_PIC
 $Comp
-L C C6
+L pic_programmer_schlib:C C6
 U 1 1 442AA12B
-P 2400 6800
-F 0 "C6" H 2450 6900 50  0000 L CNN
-F 1 "100nF" H 2450 6700 50  0000 L CNN
-F 2 "discret:C1-1" H 2750 6600 60  0000 C CNN
-F 3 "" H 2400 6800 60  0001 C CNN
-	1    2400 6800
-	1    0    0    -1
-$EndComp
-Wire Wire Line
-	2400 6200 2400 6600
+P 2400 6750
+F 0 "C6" H 2450 6850 50  0000 L CNN
+F 1 "100nF" H 2450 6650 50  0000 L CNN
+F 2 "Capacitor_THT:C_Disc_D5.1mm_W3.2mm_P5.00mm" H 2600 6600 10  0000 C CNN
+F 3 "" H 2400 6750 60  0001 C CNN
+	1    2400 6750
+	1    0    0    -1
+$EndComp
+Wire Wire Line
+	2400 6200 2400 6500
 Text Label 2750 6500 0    60   ~ 0
 VCC_PIC
 Wire Wire Line
-	5300 1500 5300 4750
+	5300 1500 5300 2100
 Connection ~ 5300 2700
 Wire Wire Line
-	5400 1400 5400 4900
+	5400 1400 5400 2000
 Connection ~ 5400 3100
 Wire Wire Line
-	10000 1500 10000 3900
+	10000 1500 10000 1900
 Connection ~ 5300 1500
 Connection ~ 10000 1900
 Wire Wire Line
-	10100 1400 10100 4000
+	10100 1400 10100 2000
 Connection ~ 10100 2000
 Connection ~ 5400 1400
 Wire Wire Line
-	10200 6200 10200 2700
-Wire Wire Line
-	5500 6200 5500 800
-Wire Wire Line
-	1900 6200 10200 6200
+	10200 6200 10200 4700
+Wire Wire Line
+	5500 6200 5500 4600
+Wire Wire Line
+	1900 6200 2100 6200
 Connection ~ 10200 4700
 Wire Wire Line
@@
 Connection ~ 5500 4600
 Wire Wire Line
-	2200 3400 2200 6300
-Wire Wire Line
-	7100 6300 1900 6300
-Wire Wire Line
-	7100 1900 7100 6300
+	2200 3400 2200 4450
+Wire Wire Line
+	7100 6300 2200 6300
+Wire Wire Line
+	7100 1900 7100 3900
 Connection ~ 2200 4450
 Connection ~ 7100 3900
@@
 	3700 1850 3700 1800
 Wire Wire Line
-	2400 7000 2400 7050
-Wire Wire Line
-	3300 7000 3300 7050
-$Comp
-L PWR_FLAG #FLG047
+	2400 6900 2400 6950
+Wire Wire Line
+	3300 6900 3300 6950
+$Comp
+L pic_programmer_schlib:PWR_FLAG #FLG047
 U 1 1 5558FA28
 P 3300 6500
@@
 	0    1    1    0
 $EndComp
+Wire Wire Line
+	2800 1200 2800 1300
+Wire Wire Line
+	2800 1300 2800 1350
+Wire Wire Line
+	5300 2700 5300 4750
+Wire Wire Line
+	5400 3100 5400 4900
+Wire Wire Line
+	5300 1500 10000 1500
+Wire Wire Line
+	10000 1900 10000 3900
+Wire Wire Line
+	10100 2000 10100 4000
+Wire Wire Line
+	5400 1400 10100 1400
+Wire Wire Line
+	10200 4700 10200 2700
+Wire Wire Line
+	5500 4600 5500 800
+Wire Wire Line
+	2200 4450 2200 6300
+Wire Wire Line
+	7100 3900 7100 6300
+Wire Wire Line
+	7200 6200 10200 6200
+Wire Wire Line
+	5500 6200 7200 6200
+Wire Wire Line
+	2200 6300 1900 6300
+Wire Wire Line
+	2100 6200 2400 6200
+Wire Wire Line
+	5400 2000 5400 3100
+Wire Wire Line
+	5300 2100 5300 2700
+Wire Wire Line
+	2400 6500 2400 6600
+Wire Wire Line
+	2400 6200 5500 6200
 $EndSCHEMATC
