File: demos/pic_programmer/pic_programmer.kicad_pcb (KiCad board)
At the start: 2 copper layers, 160 x 99.1 mm, 63 parts, among them J1 DB9-FEMAL, P1 CONN_2, P101 CONN_1, P102 CONN_1, P103 CONN_1, P104 CONN_1, P105 CONN_1, P106 CONN_1, P2 SUPP28, P3 SUPP40, Q1 BC237, Q2 BC307, Q3 BC307, U1 24Cxx, U2 74HC125, U3 7805, U4 LT1373, U5 PIC_18_PINS, U6 PIC_8_PINS

Commit message: New upstream version 5.0.0~rc1+dfsg1
Parts:
- C1, C2: footprint discret:CP10 -> Capacitors_THT:CP_Axial_L18.0mm_D6.5mm_P25.00mm_Horizontal
- C3: footprint discret:CP8 -> Capacitors_THT:C_Axial_L12.0mm_D6.5mm_P20.00mm_Horizontal
- C4, C5, C6, C7: footprint discret:C1-1 -> Capacitor_THT:C_Disc_D5.1mm_W3.2mm_P5.00mm
- C9: value 22OnF -> 220nF; footprint discret:C1-1 -> Capacitor_THT:C_Disc_D5.1mm_W3.2mm_P5.00mm
- D1, D10: footprint discret:D5 -> Diode_THT:D_DO-35_SOD27_P12.70mm_Horizontal
- D11, D2, D3, D4, D5, D6, D7: footprint discret:D3 -> Diode_THT:D_DO-35_SOD27_P7.62mm_Horizontal
- D12, D8, D9: footprint discret:LEDV -> footprints:LED_D5.0mm
- J1: footprint connect:DB9FC -> Connector_Dsub:DSUB-9_Female_Horizontal_P2.77x2.84mm_EdgePinOffset7.70mm_Housed_MountingHolesOffset9.12mm
- L1: footprint inductors:INDUCTOR_V -> footprints:INDUCTOR_V
- P1: footprint connect:bornier2 -> TerminalBlock_Phoenix:TerminalBlock_Phoenix_MKDS-1,5-2_1x02_P5.00mm_Horizontal
- P2: footprint dip_sockets:DIP-28__300_ELL -> Package_DIP:DIP-28_W7.62mm_Socket_LongPads
- P3: footprint sockets:40tex-Ell600 -> footprints:40tex-Ell600
- Q1, Q2, Q3: footprint discret:TO92 -> footprints:TO-92_BC237_307
- R1, R10, R11, R12, R13, R14, R15, R16, R17, R18, R19, R2, R20, R21, R3, R4, R5, R6, R7, R8, R9: footprint discret:R4 -> Resistor_THT:R_Axial_DIN0207_L6.3mm_D2.5mm_P10.16mm_Horizontal
- RV1: footprint discret:RV2X4 -> footprints:RV2X4
- U1, U6: footprint dip_sockets:DIP-8__300_ELL -> Package_DIP:DIP-8_W7.62mm_Socket_LongPads
- U2: footprint dip_sockets:DIP-14__300_ELL -> Package_DIP:DIP-14_W7.62mm_LongPads
- U3: footprint discret:LM78XX -> footprints:TO-220_LM78xx
- U4: footprint dip_sockets:DIP-8__300_ELL -> Package_DIP:DIP-8_W7.62mm_LongPads
- U5: footprint dip_sockets:DIP-18__300_ELL -> Package_DIP:DIP-18_W7.62mm_Socket_LongPads
- moved P2 16.9 mm to (207.6, 50.8), turned to 0 degrees
- moved C1 12.7 mm to (110.5, 78.9)
- moved C2 12.6 mm to (84.6, 90.2)
- moved U5 10.8 mm to (207.9, 108.0), turned to 0 degrees
- moved C3 10.2 mm to (134.1, 62.2)
- moved U2 8.52 mm to (115.6, 119.4), turned to 90 degrees
- moved D1 6.35 mm to (87.8, 71.1), turned to 90 degrees
- moved D10 6.35 mm to (137.2, 57.1), turned to 180 degrees
- moved J1 5.61 mm to (82.5, 121.0), turned to 270 degrees
- moved U1 5.39 mm to (179.1, 109.2), turned to 0 degrees
- moved U4 5.39 mm to (110.5, 57.1), turned to 0 degrees
- moved U6 5.39 mm to (179.1, 120.7), turned to 0 degrees
- moved R4 5.27 mm to (87.6, 107.8)
- moved R2 5.18 mm to (87.6, 114.6)
- moved R8 5.16 mm to (139.1, 91.1)
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Connections:
- net /pic_sockets/CLOCK-RB6 renamed /CLOCK-RB6
- net /pic_sockets/DATA-RB7 renamed /DATA-RB7
- net /pic_sockets/VPP-MCLR renamed /VPP/MCLR
- D1 pad 1: Net-(D1-Pad1) -> Net-(C2-Pad1)
- D1 pad 2: Net-(C2-Pad1) -> Net-(D1-Pad2)
- D10 pad 1: Net-(D10-Pad1) -> VPP
- D10 pad 2: VPP -> Net-(D10-Pad2)
- D12 pad 1: Net-(D12-Pad1) -> GND
- D12 pad 2: GND -> Net-(D12-Pad2)
- D2 pad 1: Net-(D2-Pad1) -> VCC
- D2 pad 2: VCC -> Net-(D2-Pad2)
- D3 pad 1: GND -> Net-(D2-Pad2)
- D3 pad 2: Net-(D2-Pad1) -> GND
- D4 pad 1: Net-(D4-Pad1) -> VCC
- D4 pad 2: VCC -> Net-(D4-Pad2)
- D5 pad 1: GND -> Net-(D4-Pad2)
- D5 pad 2: Net-(D4-Pad1) -> GND
- D6 pad 1: Net-(D6-Pad1) -> VCC
- D6 pad 2: VCC -> Net-(D6-Pad2)
- D7 pad 1: GND -> Net-(D6-Pad2)
- D7 pad 2: Net-(D6-Pad1) -> GND
- D8 pad 1: Net-(D8-Pad1) -> GND
- D8 pad 2: GND -> Net-(D8-Pad2)
- D9 pad 1: Net-(D9-Pad1) -> GND
- D9 pad 2: GND -> Net-(D9-Pad2)
- J1 pad 1: (no net) -> Net-(J1-Pad1)
- J1 pad 2: (no net) -> Net-(J1-Pad2)
- J1 pad 6: (no net) -> Net-(J1-Pad6)
- J1 pad 9: (no net) -> Net-(J1-Pad9)
- L1 pad 1: Net-(D10-Pad1) -> Net-(D10-Pad2)
- P1 pad 2: Net-(D1-Pad1) -> Net-(D1-Pad2)
- P101 pad 1: (no net) -> Net-(P101-Pad1)
- P102 pad 1: (no net) -> Net-(P102-Pad1)
- P103 pad 1: (no net) -> Net-(P103-Pad1)
- P104 pad 1: (no net) -> Net-(P104-Pad1)
- P105 pad 1: (no net) -> Net-(P105-Pad1)
- P106 pad 1: (no net) -> Net-(P106-Pad1)
- P2 pad 10: (no net) -> Net-(P2-Pad10)
- P2 pad 11: (no net) -> Net-(P2-Pad11)
- P2 pad 12: (no net) -> Net-(P2-Pad12)
- P2 pad 13: (no net) -> Net-(P2-Pad13)
- P2 pad 14: (no net) -> Net-(P2-Pad14)
- P2 pad 15: (no net) -> Net-(P2-Pad15)
- P2 pad 16: (no net) -> Net-(P2-Pad16)
- P2 pad 17: (no net) -> Net-(P2-Pad17)
- P2 pad 18: (no net) -> Net-(P2-Pad18)
- P2 pad 2: (no net) -> Net-(P2-Pad2)
- P2 pad 21: (no net) -> Net-(P2-Pad21)
- P2 pad 22: (no net) -> Net-(P2-Pad22)
- P2 pad 23: (no net) -> Net-(P2-Pad23)
- P2 pad 24: (no net) -> Net-(P2-Pad24)
- P2 pad 25: (no net) -> Net-(P2-Pad25)
- P2 pad 26: (no net) -> Net-(P2-Pad26)
- P2 pad 3: (no net) -> Net-(P2-Pad3)
- P2 pad 4: (no net) -> Net-(P2-Pad4)
- P2 pad 5: (no net) -> Net-(P2-Pad5)
- P2 pad 6: (no net) -> Net-(P2-Pad6)
- P2 pad 7: (no net) -> Net-(P2-Pad7)
- P2 pad 9: (no net) -> Net-(P2-Pad9)
- P3 pad 10: (no net) -> Net-(P3-Pad10)
- P3 pad 13: (no net) -> Net-(P3-Pad13)
- P3 pad 14: (no net) -> Net-(P3-Pad14)
- P3 pad 15: (no net) -> Net-(P3-Pad15)
- P3 pad 16: (no net) -> Net-(P3-Pad16)
- P3 pad 17: (no net) -> Net-(P3-Pad17)
- P3 pad 18: (no net) -> Net-(P3-Pad18)
- P3 pad 19: (no net) -> Net-(P3-Pad19)
- P3 pad 2: (no net) -> Net-(P3-Pad2)
- P3 pad 20: (no net) -> Net-(P3-Pad20)
- P3 pad 21: (no net) -> Net-(P3-Pad21)
- P3 pad 22: (no net) -> Net-(P3-Pad22)
- P3 pad 23: (no net) -> Net-(P3-Pad23)
- P3 pad 24: (no net) -> Net-(P3-Pad24)
- P3 pad 25: (no net) -> Net-(P3-Pad25)
- P3 pad 26: (no net) -> Net-(P3-Pad26)
- P3 pad 27: (no net) -> Net-(P3-Pad27)
- P3 pad 28: (no net) -> Net-(P3-Pad28)
- P3 pad 29: (no net) -> Net-(P3-Pad29)
- P3 pad 3: (no net) -> Net-(P3-Pad3)
- P3 pad 30: (no net) -> Net-(P3-Pad30)
- P3 pad 33: (no net) -> Net-(P3-Pad33)
- P3 pad 34: (no net) -> Net-(P3-Pad34)
- P3 pad 35: (no net) -> Net-(P3-Pad35)
- P3 pad 36: (no net) -> Net-(P3-Pad36)
- P3 pad 37: (no net) -> Net-(P3-Pad37)
- P3 pad 38: (no net) -> Net-(P3-Pad38)
- P3 pad 4: (no net) -> Net-(P3-Pad4)
- P3 pad 5: (no net) -> Net-(P3-Pad5)
- P3 pad 6: (no net) -> Net-(P3-Pad6)
- P3 pad 7: (no net) -> Net-(P3-Pad7)
- P3 pad 9: (no net) -> Net-(P3-Pad9)
- Q1 pad 3: Net-(D11-Pad2) -> Net-(D11-Pad1)
- R1 pad 2: Net-(D2-Pad1) -> Net-(D2-Pad2)
- R11 pad 1: Net-(D11-Pad2) -> Net-(D11-Pad1)
- R14 pad 2: Net-(D9-Pad1) -> Net-(D9-Pad2)
- R19 pad 1: Net-(D11-Pad1) -> Net-(D11-Pad2)
- R21 pad 1: Net-(D12-Pad1) -> Net-(D12-Pad2)
- R3 pad 2: Net-(D4-Pad1) -> Net-(D4-Pad2)
- R5 pad 2: Net-(D6-Pad1) -> Net-(D6-Pad2)
- R9 pad 2: Net-(D8-Pad1) -> Net-(D8-Pad2)
- U1 pad 7: (no net) -> Net-(U1-Pad7)
- U2 pad 2: Net-(D2-Pad1) -> Net-(D2-Pad2)
- U2 pad 5: Net-(D4-Pad1) -> Net-(D4-Pad2)
- U2 pad 9: Net-(D6-Pad1) -> Net-(D6-Pad2)
- U4 pad 3: (no net) -> Net-(U4-Pad3)
- U4 pad 4: (no net) -> Net-(U4-Pad4)
- U4 pad 8: Net-(D10-Pad1) -> Net-(D10-Pad2)
- U5 pad 1: (no net) -> Net-(U5-Pad1)
- U5 pad 10: (no net) -> Net-(U5-Pad10)
- U5 pad 11: (no net) -> Net-(U5-Pad11)
- U5 pad 15: (no net) -> Net-(U5-Pad15)
- U5 pad 16: (no net) -> Net-(U5-Pad16)
- U5 pad 17: (no net) -> Net-(U5-Pad17)
- U5 pad 18: (no net) -> Net-(U5-Pad18)
- U5 pad 2: (no net) -> Net-(U5-Pad2)
- U5 pad 3: (no net) -> Net-(U5-Pad3)
- U5 pad 6: (no net) -> Net-(U5-Pad6)
- U5 pad 7: (no net) -> Net-(U5-Pad7)
- U5 pad 8: (no net) -> Net-(U5-Pad8)
- U5 pad 9: (no net) -> Net-(U5-Pad9)
- U6 pad 2: (no net) -> Net-(U6-Pad2)
- U6 pad 3: (no net) -> Net-(U6-Pad3)
- U6 pad 5: (no net) -> Net-(U6-Pad5)
Routing:
- net Net-(D6-Pad2): track 0.00 -> 46.8 mm
- net Net-(D6-Pad1): track 44.0 -> 0.00 mm
- net Net-(D4-Pad2): track 0.00 -> 43.1 mm
- net Net-(D4-Pad1): track 42.7 -> 0.00 mm
- net Net-(D2-Pad2): track 0.00 -> 39.8 mm
- net Net-(D2-Pad1): track 39.4 -> 0.00 mm
- net VCC: track 183.3 -> 162.1 mm
- net Net-(D1-Pad2): track 0.00 -> 14.7 mm
- net Net-(D11-Pad1): track 5.34 -> 17.8 mm
- net Net-(D11-Pad2): track 17.3 -> 5.34 mm
- net Net-(D10-Pad2): track 0.00 -> 12.0 mm
- net Net-(D10-Pad1): track 12.0 -> 0.00 mm
- net Net-(D1-Pad1): track 10.5 -> 0.00 mm
- net Net-(Q2-Pad3): track 42.5 -> 34.5 mm
- net Net-(D12-Pad2): track 0.00 -> 6.92 mm
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
Commit message: New upstream version 5.0.0~rc2+dfsg1
Parts:
- C1, C2: footprint Capacitors_THT:CP_Axial_L18.0mm_D6.5mm_P25.00mm_Horizontal -> Capacitor_THT:CP_Axial_L18.0mm_D6.5mm_P25.00mm_Horizontal
- D12, D8, D9: footprint footprints:LED_D5.0mm -> LED_THT:LED_D5.0mm
- JP1: footprint connect:GS2 -> Jumper:SolderJumper-2_P1.3mm_Open_TrianglePad1.0x1.5mm
- L1: footprint footprints:INDUCTOR_V -> Inductor_THT:L_Radial_D7.8mm_P5.00mm_Fastron_07HCP
- P101, P102, P103, P104, P105, P106: footprint footprints:1pin-4 -> MountingHole:MountingHole_4.3mm_M4
- U3: footprint footprints:TO-220_LM78xx -> Package_TO_SOT_THT:TO-220-3_Horizontal_TabDown
- moved U3 2.54 mm to (96.5, 71.1)
- moved L1 2.54 mm to (125.7, 62.2)
- turned JP1 to 0 degrees
Routing:
- net /pic_sockets/VCC_PIC: track 292.4 -> 293.3 mm
Other:
- rule trace_min: 0.254 -> 0.25
- rule via_min_drill: 0.508 -> 0.5
- rule via_min_size: 0.889 -> 0.9

Commit message: New upstream version 5.0.0~rc3+dfsg1
Parts:
- moved J1 0.83 mm to (82.6, 120.2)
