File: demos/video/bus_pci.sch (KiCad schematic (older format))
At the start: 33 parts, among them U1 24C16, U11 S5933_PQ160

Commit message: Imported Upstream version 0.0.20070525
Connections:
- wire segments 347 -> 345
