File: demos/video/bus_pci.sch (KiCad schematic (older format))
At the start: 33 parts, among them U1 24C16, U11 S5933_PQ160

Commit message: New upstream version 5.0.0~rc1+dfsg1
Parts:
- BUS1: footprint Connect:BUSPCI -> Connectors:BUSPCI; symbol BUSPCI-5V -> video_schlib:BUSPCI-5V
- C24, C25, C26, C27, C28, C29, C30, C31: symbol C -> video_schlib:C
- C38, C67, C68, C69: symbol CP -> video_schlib:CP
- R28, R29, R5, R6, R7: symbol R -> video_schlib:R
- RR1, RR2, RR3, RR6, RR8: footprint Connect:SIL-9 -> Connectors:SIL-9; symbol RR8 -> video_schlib:RR8
- RR4, RR5, RR7: symbol RR8 -> video_schlib:RR8
- U1: symbol 24C16 -> video_schlib:24C16
- U11: symbol S5933_PQ160 -> video_schlib:S5933_PQ160
- W1, W2, W3: footprint Connect:GS2 -> Connectors:GS2; symbol TEST -> video_schlib:TEST
- W4, W5: symbol TEST -> video_schlib:TEST
