File: demos/video/graphic.sch (KiCad schematic (older format))
At the start: 34 parts, among them P10 CONN_1, P11 CONN_1, P12 CONN_1, P4 CONN_2, P5 CONN_5, P9 CONN_1, U2 4C4001, U21 XC1736APD8, U23 XC4003/PQ100, U24 XC4005-PQ160, U7 AV9173, X1 10MHz

Commit message: Imported Upstream version 0.0.20070525
Connections:
- net labels added: CCLK, DIN, DONE, PROG*
Changed lines of the file:
@@
 EESchema Schematic File Version 1
-LIBS:power,device,brooktre,linear,regul,74xx,cmos4000,adc-dac,memory,xilinx,special,analog_switches,.\video.cache
+LIBS:power,device,conn,brooktre,linear,regul,74xx,cmos4000,adc-dac,memory,xilinx,special,analog_switches,philips,.\video.cache
 EELAYER 20  0
 EELAYER END
 $Descr A3 16535 11700
 Sheet 5 8
-Title "Carte VIDEOSEQ"
-Date "19 oct 2004"
-Rev ""
-Comp ""
+Title "Video"
+Date "31 dec 2006"
+Rev "2.0B"
+Comp "Kicad EDA"
 Comment1 "Xilinxs"
 Comment2 ""
@@
 Comment4 ""
 $EndDescr
+Text Label 2400 2050 0    60   ~
+PROG*
+Text Label 3100 1900 0    60   ~
+DONE
+Text Label 3050 2000 0    60   ~
+DIN
+Text Label 3000 2200 0    60   ~
+CCLK
 Wire Wire Line
 	6150 5000 5550 5000
@@
 RESERV1
 $Comp
-L GND #PWR7
+L GND #PWR057
 U 1 1 34E1752B
 P 4850 950
-F 0 "#PWR7" H 4850 950 40  0001 C C
+F 0 "#PWR057" H 4850 950 40  0001 C C
 F 1 "GND" H 4850 880 40  0000 C C
 	1    4850 950
@@
 NoConn ~ 14100 8200
 Wire Wire Line
-	6750 5500 8200 5500
+	8200 5500 6750 5500
 Connection ~ 8200 5500
 Text Label 5600 3500 0    60   ~
@@
 NoConn ~ 5550 1700
 Wire Wire Line
-	6750 5400 6750 5500
+	6750 5500 6750 5400
 $Comp
 L XC4005-PQ100 U23
@@
 	5800 10700 5800 10650
 Wire Wire Line
-	6150 10700 6150 10650
-Wire Wire Line
-	2750 10700 6150 10700
+	6150 10650 6150 10700
+Wire Wire Line
+	6150 10700 2750 10700
 Wire Wire Line
 	5100 10250 5100 10200
@@
 	5800 10250 5800 10200
 Wire Wire Line
-	6150 10200 6150 10250
-Wire Wire Line
-	2750 10200 6150 10200
+	6150 10250 6150 10200
+Wire Wire Line
+	6150 10200 2750 10200
 Connection ~ 5800 10200
 Connection ~ 5450 10200
@@
 ACCES_RAM-
 $Comp
-L GND #PWR6
+L GND #PWR058
 U 1 1 33A80097
 P 2800 1150
-F 0 "#PWR6" H 2800 1150 40  0001 C C
+F 0 "#PWR058" H 2800 1150 40  0001 C C
 F 1 "GND" H 2800 1080 40  0000 C C
 	1    2800 1150
@@
 Connection ~ 3450 1600
 $Comp
-L VCC #PWR16
+L VCC #PWR059
 U 1 1 33A7E12B
 P 4000 1250
-F 0 "#PWR16" H 4000 1450 40  0001 C C
+F 0 "#PWR059" H 4000 1450 40  0001 C C
 F 1 "VCC" H 4000 1400 40  0000 C C
 	1    4000 1250
@@
 $EndComp
 $Comp
-L GND #PWR5
+L GND #PWR060
 U 1 1 33A7E121
 P 3700 1100
-F 0 "#PWR5" H 3700 1100 40  0001 C C
+F 0 "#PWR060" H 3700 1100 40  0001 C C
 F 1 "GND" H 3700 1030 40  0000 C C
 	1    3700 1100
@@
 	3500 1250 3450 1250
 Wire Wire Line
-	3450 1100 3500 1100
-Wire Wire Line
-	3450 1700 3450 1100
+	3500 1100 3450 1100
+Wire Wire Line
+	3450 1100 3450 1700
 Wire Wire Line
 	2900 1150 2900 2200
@@
 NoConn ~ 2500 1700
 $Comp
-L VCC #PWR15
+L VCC #PWR061
 U 1 1 33A7E07A
 P 1000 1200
-F 0 "#PWR15" H 1000 1400 40  0001 C C
+F 0 "#PWR061" H 1000 1400 40  0001 C C
 F 1 "VCC" H 1000 1350 40  0000 C C
 	1    1000 1200
@@
 Connection ~ 1000 1800
 Wire Wire Line
-	2750 1800 3450 1800
-Wire Wire Line
-	2750 2050 2750 1800
-Wire Wire Line
-	1000 2050 2750 2050
-Wire Wire Line
-	1000 1600 1000 2050
-Wire Wire Line
-	850  1400 1000 1400
-Wire Wire Line
-	850  2200 850  1400
-Wire Wire Line
-	3450 2200 850  2200
-Wire Wire Line
-	3450 2000 3000 2000
+	3450 1800 2750 1800
+Wire Wire Line
+	2750 1800 2750 2050
+Wire Wire Line
+	2750 2050 1000 2050
+Wire Wire Line
+	1000 2050 1000 1600
+Wire Wire Line
+	1000 1400 850  1400
+Wire Wire Line
+	850  1400 850  2200
+Wire Wire Line
+	850  2200 3450 2200
+Wire Wire Line
+	3000 2000 3450 2000
 Wire Wire Line
 	2500 1400 3000 1400
@@
 	2150 7300 2050 7300
 $Comp
-L VCC #PWR14
+L VCC #PWR062
 U 1 1 33A7DCF3
 P 2050 7300
-F 0 "#PWR14" H 2050 7500 40  0001 C C
+F 0 "#PWR062" H 2050 7500 40  0001 C C
 F 1 "VCC" H 2050 7450 40  0000 C C
 	1    2050 7300
@@
 	3100 7400 3100 7300
 $Comp
-L GND #PWR4
+L GND #PWR063
 U 1 1 33A7DCA9
 P 3100 7800
-F 0 "#PWR4" H 3100 7800 40  0001 C C
+F 0 "#PWR063" H 3100 7800 40  0001 C C
 F 1 "GND" H 3100 7730 40  0000 C C
 	1    3100 7800
@@
 	11300 3400 11900 3400
 $Comp
-L VCC #PWR13
+L VCC #PWR064
 U 1 1 3365FFE4
 P 8000 2150
-F 0 "#PWR13" H 8000 2350 40  0001 C C
+F 0 "#PWR064" H 8000 2350 40  0001 C C
 F 1 "VCC" H 8000 2300 40  0000 C C
 	1    8000 2150
@@
 	8000 2150 8000 2250
 Wire Wire Line
-	8000 2750 8000 2850
+	8000 2850 8000 2750
 Text GLabel 11250 7500 0    60   Output
 BLANK-
@@
 Pour CDA
 $Comp
-L GND #GND40
+L GND #GND065
 U 1 1 B3BF4EE3
 P 7400 6000
-F 0 "#GND40" H 7400 6100 60  0001 C C
+F 0 "#GND065" H 7400 6100 60  0001 C C
 F 1 "GND" H 7400 5900 60  0000 C C
 	1    7400 6000
@@
 $EndComp
 $Comp
-L GND #GND41
+L GND #GND066
 U 1 1 B3BF4EED
 P 8200 6000
-F 0 "#GND41" H 8200 6100 60  0001 C C
+F 0 "#GND066" H 8200 6100 60  0001 C C
 F 1 "GND" H 8200 5900 60  0000 C C
 	1    8200 6000
@@
 $EndComp
 $Comp
-L GND #GND42
+L GND #GND067
 U 1 1 B9ED7ABA
 P 1250 10650
-F 0 "#GND42" H 1250 10750 60  0001 C C
+F 0 "#GND067" H 1250 10750 60  0001 C C
 F 1 "GND" H 1250 10550 60  0000 C C
 	1    1250 10650
@@
 $EndComp
 $Comp
-L GND #GND43
+L GND #GND068
 U 1 1 B9ED7ABF
 P 2050 10650
-F 0 "#GND43" H 2050 10750 60  0001 C C
+F 0 "#GND068" H 2050 10750 60  0001 C C
 F 1 "GND" H 2050 10550 60  0000 C C
 	1    2050 10650
@@
 $EndComp
 $Comp
-L GND #GND44
+L GND #GND069
 U 1 1 BF805565
 P 3850 10800
-F 0 "#GND44" H 3850 10900 60  0001 C C
+F 0 "#GND069" H 3850 10900 60  0001 C C
 F 1 "GND" H 3850 10700 60  0000 C C
 	1    3850 10800
@@
 $EndComp
 $Comp
-L GND #GND45
+L GND #GND070
 U 1 1 228C46D3
 P 2750 7800
-F 0 "#GND45" H 2750 7900 60  0001 C C
+F 0 "#GND070" H 2750 7900 60  0001 C C
 F 1 "GND" H 2750 7700 60  0000 C C
 	1    2750 7800
@@
 $EndComp
 $Comp
-L GND #GND46
+L GND #GND071
 U 1 1 2295D397
 P 3350 9050
-F 0 "#GND46" H 3350 9150 60  0001 C C
+F 0 "#GND071" H 3350 9150 60  0001 C C
 F 1 "GND" H 3350 8950 60  0000 C C
 	1    3350 9050
@@
 HDREFOUT
 $Comp
-L VCC #VCC8
+L VCC #VCC072
 U 1 1 00000000
 P 2050 10150
-F 0 "#VCC8" H 2050 10350 40  0001 C C
+F 0 "#VCC072" H 2050 10350 40  0001 C C
 F 1 "VCC" H 2050 10300 40  0000 C C
 	1    2050 10150
@@
 $EndComp
 $Comp
-L VCC #VCC11
+L VCC #VCC073
 U 1 1 00000000
 P 1250 10150
-F 0 "#VCC11" H 1250 10350 40  0001 C C
+F 0 "#VCC073" H 1250 10350 40  0001 C C
 F 1 "VCC" H 1250 10300 40  0000 C C
 	1    1250 10150
@@
 $EndComp
 $Comp
-L VCC #VCC10
+L VCC #VCC074
 U 1 1 00000000
 P 11800 2800
-F 0 "#VCC10" H 11800 3000 40  0001 C C
+F 0 "#VCC074" H 11800 3000 40  0001 C C
 F 1 "VCC" H 11800 2950 40  0000 C C
 	1    11800 2800
@@
 $EndComp
 $Comp
-L VCC #VCC9
+L VCC #VCC075
 U 1 1 00000000
 P 3850 10100
-F 0 "#VCC9" H 3850 10300 40  0001 C C
+F 0 "#VCC075" H 3850 10300 40  0001 C C
 F 1 "VCC" H 3850 10250 40  0000 C C
 	1    3850 10100
@@
 	11250 4600 11900 4600
 Wire Wire Line
-	7400 4950 7500 4950
-Wire Wire Line
-	8200 4950 8000 4950
-Wire Wire Line
-	11800 3100 11900 3100
+	7500 4950 7400 4950
+Wire Wire Line
+	8000 4950 8200 4950
+Wire Wire Line
+	11900 3100 11800 3100
 Wire Wire Line
 	14100 8500 14750 8500
@@
 	2750 7300 2750 7400
 Wire Wire Line
-	2350 8650 2350 8850
-Wire Wire Line
-	2750 10650 2750 10700
+	2350 8850 2350 8650
+Wire Wire Line
+	2750 10700 2750 10650
 Wire Wire Line
 	3100 10650 3100 10700
@@
 	8200 4950 8200 5600
 Wire Wire Line
-	11800 2800 11800 3100
+	11800 3100 11800 2800
 Wire Wire Line
 	3350 7300 3350 8050
