File: demos/video/graphic.sch (KiCad schematic (older format))
At the start: 34 parts, among them P10 CONN_1, P11 CONN_1, P12 CONN_1, P4 CONN_2, P5 CONN_5, P9 CONN_1, U2 4C4001, U21 XC1736APD8, U23 XC4003/PQ100, U24 XC4005-PQ160, U7 AV9173, X1 10MHz

Commit message: Imported Upstream version 4.0.0~rc1
Parts:
- C17, C18, C19, C20, C21, C22, C23, C70, C71, C72, C73, R1, R13, R21, R26, R48: footprint (none) -> lib_smd:SM1206
- C49, C50: footprint (none) -> discret:C1
- C56: value 4,7uF -> 4.7uF; footprint (none) -> lib_smd:SM1812L
- C57: value 4,7uF -> 4.7uF; footprint (none) -> lib_smd:SM1210L
- C63: footprint (none) -> lib_smd:SM1210L
- D6: footprint (none) -> discret:LEDV
- P10, P11, P9: footprint (none) -> connect:PINTST
- P12: footprint (none) -> connect:TESTPOINT
- P4: footprint (none) -> connect:SIL-2
- P5: footprint (none) -> pin_array:PIN_ARRAY_5x1
- U2: footprint (none) -> lib_smd:SO28
- U21: footprint (none) -> dip_sockets:DIP-8__300
- U23: footprint (none) -> lib_smd:PQFP100
- U24: footprint (none) -> lib_smd:PQFP160
- U7: footprint (none) -> lib_smd:SO8E
- X1: footprint (none) -> discret:HC-18UV
Connections:
- wire segments 262 -> 277
Other:
- note added: "Decoupling"
- note added: "OSCILLATOR generates sample clock for DAC and ADC"
- note removed: "Decouplages"
- note removed: "OSCILLATEURS generation freq echantillonage CAD et CDA"
- note removed: "Pour CDA"
- moved on the sheet: C23, C63, P4, R1, R21, R48
