File: demos/video/esvideo.sch (KiCad schematic (older format))
At the start: 29 parts, among them U8 BT253, U9 BT473

Commit message: New upstream version 5.0.0~rc1+dfsg1
Parts:
- C32, C33, C34, C35, C36, C37, C39, C40, C41: symbol C -> video_schlib:C
- C42, C51, C52: symbol CP -> video_schlib:CP
- L5: symbol INDUCTOR -> video_schlib:INDUCTOR
- R15, R22, R23, R24, R36, R37, R38, R42, R43, R44, R45, R46, R47, R8: symbol R -> video_schlib:R
- U8: symbol BT253 -> video_schlib:BT253
- U9: symbol BT473 -> video_schlib:BT473
Changed lines of the file:
@@
-EESchema Schematic File Version 2
-LIBS:video_schlib
-LIBS:power
+EESchema Schematic File Version 4
 LIBS:video-cache
-EELAYER 25 0
+EELAYER 26 0
 EELAYER END
 $Descr A3 16535 11693
@@
 PCA0
 $Comp
-L GND #PWR0162
+L video_schlib:GND #PWR0162
 U 1 1 33A566EB
 P 9300 7800
@@
 Connection ~ 4350 3100
 $Comp
-L GND #PWR0163
+L video_schlib:GND #PWR0163
 U 1 1 3392D11C
 P 4350 4200
@@
 RED_IN
 $Comp
-L GND #PWR0164
+L video_schlib:GND #PWR0164
 U 1 1 335F5DFC
 P 12050 5050
@@
 $EndComp
 $Comp
-L C C32
+L video_schlib:C C32
 U 1 1 335F5DF2
 P 11800 5050
@@
 	6650 4600 6550 4600
 $Comp
-L GND #GND0165
+L video_schlib:GND #GND0165
 U 1 1 A458682C
 P 12850 4250
@@
 $EndComp
 $Comp
-L R R8
+L video_schlib:R R8
 U 1 1 A4586827
 P 12550 4250
@@
 PCA[0..2]
 $Comp
-L GND #GND0166
+L video_schlib:GND #GND0166
 U 1 1 32FA0485
 P 5650 8250
@@
 	11350 3650 13450 3650
 $Comp
-L GND #GND0167
+L video_schlib:GND #GND0167
 U 1 1 32F9F3E8
 P 10450 8250
@@
 RDCAD-
 $Comp
-L BT473 U9
+L video_schlib:BT473 U9
 U 1 1 32F9E902
 P 10350 5450
@@
 $EndComp
 $Comp
-L BT253 U8
+L video_schlib:BT253 U8
 U 1 1 32F9E7F1
 P 5500 5200
@@
 	1700 4600 1800 4600
 $Comp
-L R R42
+L video_schlib:R R42
 U 1 1 84DFB9D2
 P 12600 3000
@@
 $EndComp
 $Comp
-L R R43
+L video_schlib:R R43
 U 1 1 84DFB9D7
 P 12900 3000
@@
 $EndComp
 $Comp
-L R R44
+L video_schlib:R R44
 U 1 1 84DFB9DC
 P 13150 3000
@@
 $EndComp
 $Comp
-L C C33
+L video_schlib:C C33
 U 1 1 84DFBA31
 P 9350 2500
@@
 $EndComp
 $Comp
-L C C34
+L video_schlib:C C34
 U 1 1 84DFBA36
 P 11650 2600
@@
 $EndComp
 $Comp
-L CP C42
+L video_schlib:CP C42
 U 1 1 84DFBAEF
 P 12150 2600
@@
 $EndComp
 $Comp
-L C C35
+L video_schlib:C C35
 U 1 1 84DFBB21
 P 11450 3100
@@
 $EndComp
 $Comp
-L GND #GND0168
+L video_schlib:GND #GND0168
 U 1 1 684863B9
 P 9350 2750
@@
 $EndComp
 $Comp
-L GND #GND0169
+L video_schlib:GND #GND0169
 U 1 1 684863BE
 P 9850 2750
@@
 $EndComp
 $Comp
-L GND #GND0170
+L video_schlib:GND #GND0170
 U 1 1 684863C3
 P 12600 2700
@@
 $EndComp
 $Comp
-L GND #GND0171
+L video_schlib:GND #GND0171
 U 1 1 684863C8
 P 12900 2700
@@
 $EndComp
 $Comp
-L GND #GND0172
+L video_schlib:GND #GND0172
 U 1 1 684863CD
 P 13150 2700
@@
 $EndComp
 $Comp
-L GND #GND0173
+L video_schlib:GND #GND0173
 U 1 1 A44C032A
 P 6650 4400
@@
 $EndComp
 $Comp
-L R R47
+L video_schlib:R R47
 U 1 1 A44C0348
 P 2050 5000
@@
 $EndComp
 $Comp
-L R R45
+L video_schlib:R R45
 U 1 1 A44C032F
 P 2050 5800
@@
 $EndComp
 $Comp
-L R R46
+L video_schlib:R R46
 U 1 1 A44C0339
 P 2050 6600
@@
 $EndComp
 $Comp
-L GND #GND0174
+L video_schlib:GND #GND0174
 U 1 1 A44C0393
 P 2350 5000
@@
 $EndComp
 $Comp
-L GND #GND0175
+L video_schlib:GND #GND0175
 U 1 1 A44C0398
 P 2350 5800
@@
 $EndComp
 $Comp
-L GND #GND0176
+L video_schlib:GND #GND0176
 U 1 1 A44C039D
 P 2350 6600
@@
 $EndComp
 $Comp
-L R R38
+L video_schlib:R R38
 U 1 1 A44C03AC
 P 4100 2900
@@
 $EndComp
 $Comp
-L GND #GND0177
+L video_schlib:GND #GND0177
 U 1 1 A44C03B1
 P 3800 2900
@@
 $EndComp
 $Comp
-L GND #GND0178
+L video_schlib:GND #GND0178
 U 1 1 A44D982F
 P 3800 1450
@@
 $EndComp
 $Comp
-L R R15
+L video_schlib:R R15
 U 1 1 A44D982A
 P 3800 1750
@@
 $EndComp
 $Comp
-L GND #GND0179
+L video_schlib:GND #GND0179
 U 1 1 A44D9852
 P 3300 2800
@@
 $EndComp
 $Comp
-L C C36
+L video_schlib:C C36
 U 1 1 A44D9848
 P 3800 2400
@@
 $EndComp
 $Comp
-L R R36
+L video_schlib:R R36
 U 1 1 A44D9843
 P 4100 2800
@@
 $EndComp
 $Comp
-L C C37
+L video_schlib:C C37
 U 1 1 A44D984D
 P 3550 2800
@@
 $EndComp
 $Comp
-L R R24
+L video_schlib:R R24
 U 1 1 A44C034D
 P 2050 4600
@@
 $EndComp
 $Comp
-L R R23
+L video_schlib:R R23
 U 1 1 A44C0343
 P 2050 5400
@@
 $EndComp
 $Comp
-L R R22
+L video_schlib:R R22
 U 1 1 A44C0334
 P 2050 6200
@@
 $EndComp
 $Comp
-L C C39
+L video_schlib:C C39
 U 1 1 A44C037F
 P 2550 4600
@@
 $EndComp
 $Comp
-L C C40
+L video_schlib:C C40
 U 1 1 A44C0384
 P 2550 5400
@@
 $EndComp
 $Comp
-L C C41
+L video_schlib:C C41
 U 1 1 A44C0389
 P 2550 6200
@@
 $EndComp
 $Comp
-L GND #GND0180
+L video_schlib:GND #GND0180
 U 1 1 26FC0C80
 P 6400 2200
@@
 $EndComp
 $Comp
-L CP C52
+L video_schlib:CP C52
 U 1 1 84DFB9B9
 P 6150 2200
@@
 $EndComp
 $Comp
-L CP C51
+L video_schlib:CP C51
 U 1 1 28ED6A43
 P 9850 2500
@@
 $EndComp
 $Comp
-L INDUCTOR L5
+L video_schlib:INDUCTOR L5
 U 1 1 84DFBB99
 P 12150 1800
@@
 $EndComp
 $Comp
-L R R37
+L video_schlib:R R37
 U 1 1 5D7688E4
 P 3700 3100
@@
 $EndComp
 $Comp
-L GND #GND0181
+L video_schlib:GND #GND0181
 U 1 1 5D7688FD
 P 3400 3100
@@
 REF+
 $Comp
-L VCC #VCC0182
+L video_schlib:VCC #VCC0182
 U 1 1 4BF036B4
 P 12150 1450
