File: demos/video/muxdata.sch (KiCad schematic (older format))
At the start: 5 parts, among them U22 XC4003-VQ100, U3 74LS245, U4 74LS245, U5 74LS245, U6 74LS245

Commit message: Imported Upstream version 4.0.0~rc1
Parts:
- U22: footprint (none) -> lib_smd:VQFP100
- U3, U4, U5, U6: footprint (none) -> lib_smd:SO20L
Other:
- moved on the sheet: U22, U3, U4, U5, U6
