File: demos/video/muxdata.sch (KiCad schematic (older format))
At the start: 5 parts, among them U22 XC4003-VQ100, U3 74LS245, U4 74LS245, U5 74LS245, U6 74LS245

Commit message: New upstream version 5.0.0~rc1+dfsg1
Parts:
- U22: symbol XC4003-VQ100 -> video_schlib:XC4003-VQ100
- U3, U4, U5, U6: symbol 74LS245 -> video_schlib:74LS245
Changed lines of the file:
@@
-EESchema Schematic File Version 2
-LIBS:video_schlib
-LIBS:power
+EESchema Schematic File Version 4
 LIBS:video-cache
-EELAYER 25 0
+EELAYER 26 0
 EELAYER END
 $Descr A4 11693 8268
@@
 VRAM0
 $Comp
-L 74LS245 U6
+L video_schlib:74LS245 U6
 U 1 1 4BF036D5
 P 3300 5200
@@
 $EndComp
 $Comp
-L 74LS245 U5
+L video_schlib:74LS245 U5
 U 1 1 4BF036D6
 P 3300 4000
@@
 $EndComp
 $Comp
-L 74LS245 U4
+L video_schlib:74LS245 U4
 U 1 1 4BF036D7
 P 3300 2800
@@
 $EndComp
 $Comp
-L 74LS245 U3
+L video_schlib:74LS245 U3
 U 1 1 33A7E303
 P 3300 1600
@@
 VRAM[0..31]
 $Comp
-L VCC #PWR06
+L video_schlib:VCC #PWR06
 U 1 1 33A567E7
 P 6100 1550
@@
 	6100 1800 6100 1550
 $Comp
-L XC4003-VQ100 U22
+L video_schlib:XC4003-VQ100 U22
 U 1 1 33A567B8
 P 7050 3850
