File: demos/video/pal-ntsc.sch (KiCad schematic (older format))
At the start: 36 parts, among them U10 BT812, X2 30MHz

Commit message: Imported Upstream version 4.0.0~rc1
Parts:
- C1, C10, C11, C12, C13, C14, C15, C16, C2, C3, C4, C47, C5, C6, C65, C66, C7, C8, C9, R12, R14, R19, R2, R20, R25, R27, R3, R35: footprint (none) -> lib_smd:SM1206
- C62: footprint (none) -> lib_smd:SM1210L
- D1, D2, D3, D4: footprint (none) -> discret:D3
- L4: footprint (none) -> lib_smd:SM1812
- U10: footprint (none) -> lib_smd:PQFP160
- X2: footprint (none) -> discret:HC-18UV
Other:
- moved on the sheet: C47, R14, R19
