File: demos/video/pal-ntsc.sch (KiCad schematic (older format))
At the start: 36 parts, among them U10 BT812, X2 30MHz

Commit message: New upstream version 5.0.0~rc1+dfsg1
Parts:
- C1, C10, C11, C12, C13, C14, C15, C16, C2, C3, C4, C47, C5, C6, C65, C66, C7, C8, C9: symbol C -> video_schlib:C
- C62: symbol CP -> video_schlib:CP
- D1, D2, D3, D4: symbol DIODESCH -> video_schlib:DIODESCH
- L4: symbol INDUCTOR -> video_schlib:INDUCTOR
- R12, R14, R19, R2, R20, R25, R27, R3, R35: symbol R -> video_schlib:R
- U10: symbol BT812 -> video_schlib:BT812
- X2: symbol CRYSTAL -> video_schlib:CRYSTAL
Changed lines of the file:
@@
-EESchema Schematic File Version 2
-LIBS:video_schlib
-LIBS:power
+EESchema Schematic File Version 4
 LIBS:video-cache
-EELAYER 25 0
+EELAYER 26 0
 EELAYER END
 $Descr A3 16535 11693
@@
 BT812_RD-
 $Comp
-L VCC #VCC034
+L video_schlib:VCC #VCC034
 U 1 1 4BF036C7
 P 6350 2300
@@
 NoConn ~ 10050 7700
 $Comp
-L INDUCTOR L4
+L video_schlib:INDUCTOR L4
 U 1 1 811D9080
 P 10150 1800
@@
 $EndComp
 $Comp
-L GND #GND035
+L video_schlib:GND #GND035
 U 1 1 821CDA95
 P 4000 7250
@@
 $EndComp
 $Comp
-L GND #GND036
+L video_schlib:GND #GND036
 U 1 1 821CDAA4
 P 3200 7050
@@
 $EndComp
 $Comp
-L R R35
+L video_schlib:R R35
 U 1 1 821CDAB8
 P 2800 6500
@@
 $EndComp
 $Comp
-L C C1
+L video_schlib:C C1
 U 1 1 821CDAC2
 P 3500 6500
@@
 $EndComp
 $Comp
-L GND #GND037
+L video_schlib:GND #GND037
 U 1 1 A9C8254A
 P 6350 9900
@@
 $EndComp
 $Comp
-L GND #GND038
+L video_schlib:GND #GND038
 U 1 1 A9C8254F
 P 8950 9900
@@
 $EndComp
 $Comp
-L GND #GND039
+L video_schlib:GND #GND039
 U 1 1 A9C82559
 P 5950 6200
@@
 $EndComp
 $Comp
-L GND #GND040
+L video_schlib:GND #GND040
 U 1 1 A9C8255E
 P 5950 6000
@@
 $EndComp
 $Comp
-L GND #GND041
+L video_schlib:GND #GND041
 U 1 1 A9C82563
 P 5950 6600
@@
 $EndComp
 $Comp
-L GND #GND042
+L video_schlib:GND #GND042
 U 1 1 A9CA7F70
 P 11950 3600
@@
 $EndComp
 $Comp
-L C C2
+L video_schlib:C C2
 U 1 1 A9CA7F6B
 P 11950 3250
@@
 $EndComp
 $Comp
-L C C3
+L video_schlib:C C3
 U 1 1 A9CA7F75
 P 3450 4200
@@
 $EndComp
 $Comp
-L C C4
+L video_schlib:C C4
 U 1 1 A9CA7F7A
 P 3450 5100
@@
 $EndComp
 $Comp
-L R R14
+L video_schlib:R R14
 U 1 1 821CDA9A
 P 4000 6950
@@
 $EndComp
 $Comp
-L R R3
+L video_schlib:R R3
 U 1 1 8116F4AA
 P 4100 4200
@@
 $EndComp
 $Comp
-L R R2
+L video_schlib:R R2
 U 1 1 8116F4A5
 P 4100 5100
@@
 $EndComp
 $Comp
-L DIODESCH D1
+L video_schlib:DIODESCH D1
 U 1 1 A9CA7F7F
 P 3850 3700
@@
 $EndComp
 $Comp
-L DIODESCH D2
+L video_schlib:DIODESCH D2
 U 1 1 A9CA7F84
 P 3850 3300
@@
 $EndComp
 $Comp
-L DIODESCH D3
+L video_schlib:DIODESCH D3
 U 1 1 A9CA7F8E
 P 4050 6000
@@
 $EndComp
 $Comp
-L DIODESCH D4
+L video_schlib:DIODESCH D4
 U 1 1 A9CA7F93
 P 4050 5600
@@
 $EndComp
 $Comp
-L GND #GND043
+L video_schlib:GND #GND043
 U 1 1 A9CA7F9D
 P 3850 6000
@@
 $EndComp
 $Comp
-L GND #GND044
+L video_schlib:GND #GND044
 U 1 1 A9CA7FA2
 P 3600 3700
@@
 $EndComp
 $Comp
-L GND #GND045
+L video_schlib:GND #GND045
 U 1 1 A9CA7FBB
 P 5200 6100
@@
 $EndComp
 $Comp
-L GND #GND046
+L video_schlib:GND #GND046
 U 1 1 A9CA7FC0
 P 4650 6400
@@
 $EndComp
 $Comp
-L R R27
+L video_schlib:R R27
 U 1 1 A9CA7FC5
 P 5500 6800
@@
 $EndComp
 $Comp
-L R R12
+L video_schlib:R R12
 U 1 1 A9CA7FCA
 P 5200 7100
@@
 $EndComp
 $Comp
-L C C65
+L video_schlib:C C65
 U 1 1 B15DA8C5
 P 4850 1700
@@
 $EndComp
 $Comp
-L C C66
+L video_schlib:C C66
 U 1 1 B15DA8CA
 P 5650 1700
@@
 $EndComp
 $Comp
-L GND #GND047
+L video_schlib:GND #GND047
 U 1 1 B15DA8CF
 P 4850 1450
@@
 $EndComp
 $Comp
-L GND #GND048
+L video_schlib:GND #GND048
 U 1 1 B15DA8D4
 P 5650 1450
@@
 $EndComp
 $Comp
-L GND #GND049
+L video_schlib:GND #GND049
 U 1 1 B175430E
 P 5800 4100
@@
 $EndComp
 $Comp
-L CRYSTAL X2
+L video_schlib:CRYSTAL X2
 U 1 1 B15DA8C0
 P 5250 2100
@@
 $EndComp
 $Comp
-L R R19
+L video_schlib:R R19
 U 1 1 A9CA7FA7
 P 11050 6200
@@
 $EndComp
 $Comp
-L C C5
+L video_schlib:C C5
 U 1 1 A9CA7FAC
 P 11650 6200
@@
 $EndComp
 $Comp
-L R R20
+L video_schlib:R R20
 U 1 1 B176B9C3
 P 11100 5800
@@
 $EndComp
 $Comp
-L C C8
+L video_schlib:C C8
 U 1 1 B176B9C8
 P 11650 5800
@@
 $EndComp
 $Comp
-L C C6
+L video_schlib:C C6
 U 1 1 A9CA7FB1
 P 5450 6100
@@
 $EndComp
 $Comp
-L C C7
+L video_schlib:C C7
 U 1 1 A9CA7FB6
 P 4900 6400
@@
 $EndComp
 $Comp
-L C C47
+L video_schlib:C C47
 U 1 1 821CDABD
 P 3200 6800
@@
 $EndComp
 $Comp
-L BT812 U10
+L video_schlib:BT812 U10
 U 1 1 BECCB834
 P 8000 6100
@@
 $EndComp
 $Comp
-L CP C62
+L video_schlib:CP C62
 U 1 1 811D9071
 P 10750 2300
@@
 $EndComp
 $Comp
-L GND #GND050
+L video_schlib:GND #GND050
 U 1 1 BF69A158
 P 10750 2550
@@
 $EndComp
 $Comp
-L GND #GND051
+L video_schlib:GND #GND051
 U 1 1 BF69A16C
 P 13050 9200
@@
 $EndComp
 $Comp
-L C C9
+L video_schlib:C C9
 U 1 1 BF69A15D
 P 13050 8850
@@
 $EndComp
 $Comp
-L C C10
+L video_schlib:C C10
 U 1 1 BF69A162
 P 13750 8850
@@
 $EndComp
 $Comp
-L C C11
+L video_schlib:C C11
 U 1 1 BF69A167
 P 14450 8850
@@
 $EndComp
 $Comp
-L C C14
+L video_schlib:C C14
 U 1 1 BF69A17B
 P 14050 3250
@@
 $EndComp
 $Comp
-L C C13
+L video_schlib:C C13
 U 1 1 BF69A176
 P 13350 3250
@@
 $EndComp
 $Comp
-L C C12
+L video_schlib:C C12
 U 1 1 BF69A171
 P 12650 3250
@@
 $EndComp
 $Comp
-L GND #GND052
+L video_schlib:GND #GND052
 U 1 1 0F47DCBD
 P 10250 9600
@@
 $EndComp
 $Comp
-L C C16
+L video_schlib:C C16
 U 1 1 0F47DCB8
 P 10250 9350
@@
 $EndComp
 $Comp
-L R R25
+L video_schlib:R R25
 U 1 1 B1754313
 P 5300 2600
@@
 PC_A1
 $Comp
-L VCC #VCC053
+L video_schlib:VCC #VCC053
 U 1 1 4BF036C8
 P 13050 8500
@@
 $EndComp
 $Comp
-L VCC #VCC054
+L video_schlib:VCC #VCC054
 U 1 1 4BF036C9
 P 9750 1800
@@
 $EndComp
 $Comp
-L VCC #VCC055
+L video_schlib:VCC #VCC055
 U 1 1 4BF036CA
 P 3850 5600
@@
 $EndComp
 $Comp
-L VCC #VCC056
+L video_schlib:VCC #VCC056
 U 1 1 00000000
 P 3600 3300
@@
 Connection ~ 14450 9100
 $Comp
-L C C15
+L video_schlib:C C15
 U 1 1 0939A342
 P 15150 8850
