File: demos/video/rams.sch (KiCad schematic (older format))
At the start: 8 parts, among them U12 SIM4X32, U13 SIM4X32, U14 SIM4X32, U15 SIM4X32, U16 SIM4X32, U17 SIM4X32, U18 SIM4X32, U19 SIM4X32

Commit message: Imported Upstream version 4.0.0~rc1
Parts:
- U12, U13, U14, U15, U16, U17, U18, U19: footprint (none) -> footprints:sim72
Other:
- moved on the sheet: U12, U13, U14, U15, U16, U17, U18, U19
