File: demos/video/rams.sch (KiCad schematic (older format))
At the start: 8 parts, among them U12 SIM4X32, U13 SIM4X32, U14 SIM4X32, U15 SIM4X32, U16 SIM4X32, U17 SIM4X32, U18 SIM4X32, U19 SIM4X32

Commit message: New upstream version 5.0.0~rc1+dfsg1
Parts:
- U12, U13, U14, U15, U16, U17, U18, U19: symbol SIM4X32 -> video_schlib:SIM4X32
Changed lines of the file:
@@
-EESchema Schematic File Version 2
-LIBS:video_schlib
-LIBS:power
+EESchema Schematic File Version 4
 LIBS:video-cache
-EELAYER 25 0
+EELAYER 26 0
 EELAYER END
 $Descr A3 16535 11693
@@
 MXA0
 $Comp
-L SIM4X32 U13
+L video_schlib:SIM4X32 U13
 U 1 1 32FA1E5B
 P 12100 7450
@@
 MXA0
 $Comp
-L SIM4X32 U14
+L video_schlib:SIM4X32 U14
 U 1 1 4BF036CF
 P 9300 7450
@@
 MXA0
 $Comp
-L SIM4X32 U12
+L video_schlib:SIM4X32 U12
 U 1 1 4BF036CE
 P 6450 7450
@@
 MXA0
 $Comp
-L SIM4X32 U16
+L video_schlib:SIM4X32 U16
 U 1 1 4BF036D0
 P 3600 7450
@@
 MXA0
 $Comp
-L SIM4X32 U15
+L video_schlib:SIM4X32 U15
 U 1 1 4BF036D1
 P 12100 3000
@@
 MXA0
 $Comp
-L SIM4X32 U17
+L video_schlib:SIM4X32 U17
 U 1 1 4BF036D2
 P 9300 3000
@@
 MXA0
 $Comp
-L SIM4X32 U18
+L video_schlib:SIM4X32 U18
 U 1 1 4BF036D3
 P 6450 3000
@@
 MXA0
 $Comp
-L SIM4X32 U19
+L video_schlib:SIM4X32 U19
 U 1 1 4BF036D4
 P 3600 3000
