File: demos/video/video.sch (KiCad schematic (older format))
At the start: 5 parts, among them J4 DB9FEM, P1 BNC, P2 BNC, P3 BNC, P8 BNC

Commit message: Imported Upstream version 4.0.0~rc1
Parts:
- J4: footprint (none) -> connect:DB9FC
- P1, P2, P3, P8: footprint (none) -> discret:SUBCLICK
Connections:
- wire segments 147 -> 144
Other:
- moved on the sheet: J4, P1, P2, P3, P8
