File: demos/video/video.sch (KiCad schematic (older format))
At the start: 5 parts, among them J4 DB9FEM, P1 BNC, P2 BNC, P3 BNC, P8 BNC

Commit message: New upstream version 5.0.0~rc1+dfsg1
Parts:
- J4: footprint Connect:DB9FC -> Connectors:DB9FC; symbol DB9 -> video_schlib:DB9
- P1, P2, P3, P8: symbol BNC -> video_schlib:BNC
Changed lines of the file:
@@
-EESchema Schematic File Version 2
-LIBS:video_schlib
-LIBS:power
+EESchema Schematic File Version 4
 LIBS:video-cache
-EELAYER 25 0
+EELAYER 26 0
 EELAYER END
 $Descr A3 16535 11693
@@
 	8850 2750 9500 2750
 $Comp
-L GND #GND01
+L video_schlib:GND #GND01
 U 1 1 84DFBB6C
 P 14800 4650
@@
 $EndComp
 $Comp
-L DB9 J4
+L video_schlib:DB9 J4
 U 1 1 84DFBB8F
 P 15350 4050
 F 0 "J4" H 15350 4600 70  0000 C CNN
 F 1 "DB9FEM" H 15350 3500 70  0000 C CNN
-F 2 "Connect:DB9FC" H 15350 4050 60  0001 C CNN
+F 2 "Connectors:DB9FC" H 15350 4050 60  0001 C CNN
 F 3 "" H 15350 4050 60  0001 C CNN
 	1    15350 4050
@@
 	14650 1900 15200 1900
 $Comp
-L GND #GND02
+L video_schlib:GND #GND02
 U 1 1 30705D34
 P 15350 2900
@@
 $EndComp
 $Comp
-L BNC P8
+L video_schlib:BNC P8
 U 1 1 30705D02
 P 15350 2700
@@
 RED_IN
 $Comp
-L GND #GND03
+L video_schlib:GND #GND03
 U 1 1 32FA02CD
 P 12100 2800
@@
 $EndComp
 $Comp
-L GND #GND04
+L video_schlib:GND #GND04
 U 1 1 32FA02C6
 P 12100 3600
@@
 $EndComp
 $Comp
-L GND #GND05
+L video_schlib:GND #GND05
 U 1 1 32FA02C2
 P 12100 2000
@@
 $EndComp
 $Comp
-L BNC P3
+L video_schlib:BNC P3
 U 1 1 32F9F1AD
 P 12100 3400
@@
 $EndComp
 $Comp
-L BNC P2
+L video_schlib:BNC P2
 U 1 1 32F9F1A3
 P 12100 2600
@@
 $EndComp
 $Comp
-L BNC P1
+L video_schlib:BNC P1
 U 1 1 32F9F198
 P 12100 1800
