File: demos/video/modul.sch (KiCad schematic (older format))
At the start: 39 parts, among them Q1 BC848, Q2 BC848, Q3 BC848, U20 TDA8501, X3 4.433618MHz

Commit message: New upstream version 5.0.0~rc1+dfsg1
Parts:
- C43, C44, C45, C46, C48, C53, C58, C59, C60, C61: symbol C -> video_schlib:C
- C54, C55, C64: symbol CP -> video_schlib:CP
- CV1: symbol CTRIM -> video_schlib:CTRIM
- L1, L2, L3: symbol INDUCTOR -> video_schlib:INDUCTOR
- L6: symbol LIGNE_A_RETARD -> video_schlib:LIGNE_A_RETARD
- POT1: symbol POT -> video_schlib:POT
- Q1, Q2, Q3: symbol NPN -> video_schlib:NPN
- R10, R11, R16, R17, R18, R30, R31, R32, R33, R34, R39, R4, R40, R41, R9: symbol R -> video_schlib:R
- U20: symbol TDA8501 -> video_schlib:TDA8501
- X3: symbol CRYSTAL -> video_schlib:CRYSTAL
Changed lines of the file:
@@
-EESchema Schematic File Version 2
-LIBS:video_schlib
-LIBS:power
+EESchema Schematic File Version 4
 LIBS:video-cache
-EELAYER 25 0
+EELAYER 26 0
 EELAYER END
 $Descr A4 11693 8268
@@
 	6900 1200 7300 1200
 $Comp
-L PWR_FLAG #FLG07
+L video_schlib:PWR_FLAG #FLG07
 U 1 1 4174D92E
 P 3500 1450
@@
 $EndComp
 $Comp
-L PWR_FLAG #FLG08
+L video_schlib:PWR_FLAG #FLG08
 U 1 1 4174D923
 P 6900 1200
@@
 	5100 2400 5350 2400
 $Comp
-L GND #PWR09
+L video_schlib:GND #PWR09
 U 1 1 349FB5CD
 P 5650 2600
@@
 	4400 2700 6900 2700
 $Comp
-L LIGNE_A_RETARD L6
+L video_schlib:LIGNE_A_RETARD L6
 U 1 1 349FB562
 P 5650 2400
@@
 $EndComp
 $Comp
-L GND #PWR010
+L video_schlib:GND #PWR010
 U 1 1 33CF5737
 P 4450 3800
@@
 	1950 3300 2000 3300
 $Comp
-L VCC #PWR011
+L video_schlib:VCC #PWR011
 U 1 1 33A51A5E
 P 1950 3300
@@
 $EndComp
 $Comp
-L R R4
+L video_schlib:R R4
 U 1 1 33A51A4E
 P 2250 3300
@@
 3.579545MHz
 $Comp
-L GND #GND012
+L video_schlib:GND #GND012
 U 1 1 22760F6C
 P 3500 4500
@@
 $EndComp
 $Comp
-L GND #GND013
+L video_schlib:GND #GND013
 U 1 1 22760F7B
 P 3900 2050
@@
 $EndComp
 $Comp
-L GND #GND014
+L video_schlib:GND #GND014
 U 1 1 22760F94
 P 1500 4400
@@
 $EndComp
 $Comp
-L GND #GND015
+L video_schlib:GND #GND015
 U 1 1 22760F9E
 P 950 3900
@@
 $EndComp
 $Comp
-L GND #GND016
+L video_schlib:GND #GND016
 U 1 1 22760FAD
 P 2100 5600
@@
 $EndComp
 $Comp
-L GND #GND017
+L video_schlib:GND #GND017
 U 1 1 22760FC6
 P 6300 3300
@@
 $EndComp
 $Comp
-L GND #GND018
+L video_schlib:GND #GND018
 U 1 1 22760FD0
 P 5200 3500
@@
 $EndComp
 $Comp
-L GND #GND019
+L video_schlib:GND #GND019
 U 1 1 22760FDA
 P 4500 4450
@@
 $EndComp
 $Comp
-L GND #GND020
+L video_schlib:GND #GND020
 U 1 1 22760FE9
 P 3300 1850
@@
 $EndComp
 $Comp
-L GND #GND021
+L video_schlib:GND #GND021
 U 1 1 22761002
 P 5500 5150
@@
 $EndComp
 $Comp
-L GND #GND022
+L video_schlib:GND #GND022
 U 1 1 22761007
 P 6200 5150
@@
 $EndComp
 $Comp
-L GND #GND023
+L video_schlib:GND #GND023
 U 1 1 2276104D
 P 9800 2150
@@
 $EndComp
 $Comp
-L GND #GND024
+L video_schlib:GND #GND024
 U 1 1 2276105C
 P 7200 1750
@@
 $EndComp
 $Comp
-L GND #GND025
+L video_schlib:GND #GND025
 U 1 1 2276106B
 P 9800 3750
@@
 $EndComp
 $Comp
-L GND #GND026
+L video_schlib:GND #GND026
 U 1 1 22761084
 P 9800 5350
@@
 $EndComp
 $Comp
-L GND #GND027
+L video_schlib:GND #GND027
 U 1 1 227610A2
 P 6800 3950
@@
 CVBS
 $Comp
-L VCC #VCC028
+L video_schlib:VCC #VCC028
 U 1 1 4BF036B3
 P 4700 1500
@@
 $EndComp
 $Comp
-L +5F #+029
+L video_schlib:+5F #+029
 U 1 1 4BF036B2
 P 9800 900
@@
 $EndComp
 $Comp
-L +5F #+030
+L video_schlib:+5F #+030
 U 1 1 4BF036B1
 P 7100 1100
@@
 $EndComp
 $Comp
-L +5F #+031
+L video_schlib:+5F #+031
 U 1 1 4BF036B0
 P 9800 2500
@@
 $EndComp
 $Comp
-L +5F #+032
+L video_schlib:+5F #+032
 U 1 1 4BF0369E
 P 9800 4100
@@
 	6800 3600 6600 3600
 $Comp
-L POT POT1
+L video_schlib:POT POT1
 U 1 1 2276109D
 P 6350 3600
@@
 COUT
 $Comp
-L VCC #VCC033
+L video_schlib:VCC #VCC033
 U 1 1 4BF0369D
 P 8000 1200
@@
 	7900 1200 8000 1200
 $Comp
-L NPN Q1
+L video_schlib:NPN Q1
 U 1 1 22761039
 P 9700 1200
@@
 $EndComp
 $Comp
-L NPN Q2
+L video_schlib:NPN Q2
 U 1 1 22761066
 P 9700 2800
@@
 $EndComp
 $Comp
-L NPN Q3
+L video_schlib:NPN Q3
 U 1 1 2276107F
 P 9700 4400
@@
 $EndComp
 $Comp
-L CP C54
+L video_schlib:CP C54
 U 1 1 22760F76
 P 3900 1800
@@
 $EndComp
 $Comp
-L R R39
+L video_schlib:R R39
 U 1 1 22761048
 P 10250 1500
@@
 $EndComp
 $Comp
-L R R16
+L video_schlib:R R16
 U 1 1 2276103E
 P 9150 1200
@@
 $EndComp
 $Comp
-L R R17
+L video_schlib:R R17
 U 1 1 2276107A
 P 9150 2800
@@
 $EndComp
 $Comp
-L R R40
+L video_schlib:R R40
 U 1 1 22761075
 P 10250 3100
@@
 $EndComp
 $Comp
-L R R18
+L video_schlib:R R18
 U 1 1 22761093
 P 9150 4400
@@
 $EndComp
 $Comp
-L R R41
+L video_schlib:R R41
 U 1 1 2276108E
 P 10250 4700
@@
 Connection ~ 9800 1500
 $Comp
-L R R30
+L video_schlib:R R30
 U 1 1 22760FE4
 P 2150 1800
@@
 $EndComp
 $Comp
-L R R31
+L video_schlib:R R31
 U 1 1 22760FDF
 P 2950 1800
@@
 $EndComp
 $Comp
-L R R10
+L video_schlib:R R10
 U 1 1 22760F80
 P 4850 2400
@@
 $EndComp
 $Comp
-L R R11
+L video_schlib:R R11
 U 1 1 22760FBC
 P 6550 3000
@@
 $EndComp
 $Comp
-L R R9
+L video_schlib:R R9
 U 1 1 22761098
 P 5750 3600
@@
 $EndComp
 $Comp
-L C C61
+L video_schlib:C C61
 U 1 1 22760F8A
 P 2500 2150
@@
 $EndComp
 $Comp
-L C C60
+L video_schlib:C C60
 U 1 1 22760F67
 P 2300 3500
@@
 $EndComp
 $Comp
-L C C43
+L video_schlib:C C43
 U 1 1 22760F8F
 P 1500 4150
@@
 $EndComp
 $Comp
-L CTRIM CV1
+L video_schlib:CTRIM CV1
 U 1 1 22760FA8
 P 2100 5350
@@
 $EndComp
 $Comp
-L C C45
+L video_schlib:C C45
 U 1 1 22760FD5
 P 4500 4200
@@
 $EndComp
 $Comp
-L C C48
+L video_schlib:C C48
 U 1 1 22760FCB
 P 5200 3300
@@
 $EndComp
 $Comp
-L CP C64
+L video_schlib:CP C64
 U 1 1 22760FC1
 P 6100 3300
@@
 $EndComp
 $Comp
-L C C44
+L video_schlib:C C44
 U 1 1 22760F99
 P 950 3650
@@
 CSYNC-OUT
 $Comp
-L C C53
+L video_schlib:C C53
 U 1 1 22760FF8
 P 5500 4900
@@
 $EndComp
 $Comp
-L INDUCTOR L1
+L video_schlib:INDUCTOR L1
 U 1 1 22760FF3
 P 5500 4200
@@
 $EndComp
 $Comp
-L INDUCTOR L3
+L video_schlib:INDUCTOR L3
 U 1 1 22761052
 P 7600 1200
@@
 $EndComp
 $Comp
-L INDUCTOR L2
+L video_schlib:INDUCTOR L2
 U 1 1 22760F71
 P 4300 1500
@@
 $EndComp
 $Comp
-L TDA8501 U20
+L video_schlib:TDA8501 U20
 U 1 1 22760F4E
 P 3500 3400
@@
 $EndComp
 $Comp
-L C C46
+L video_schlib:C C46
 U 1 1 22760FFD
 P 6200 4900
@@
 $EndComp
 $Comp
-L R R34
+L video_schlib:R R34
 U 1 1 22761089
 P 9800 5050
@@
 $EndComp
 $Comp
-L R R33
+L video_schlib:R R33
 U 1 1 22761070
 P 9800 3450
@@
 $EndComp
 $Comp
-L R R32
+L video_schlib:R R32
 U 1 1 22761043
 P 9800 1850
@@
 $EndComp
 $Comp
-L CP C55
+L video_schlib:CP C55
 U 1 1 22761057
 P 7200 1500
@@
 $EndComp
 $Comp
-L C C59
+L video_schlib:C C59
 U 1 1 22760F62
 P 1800 3600
@@
 $EndComp
 $Comp
-L C C58
+L video_schlib:C C58
 U 1 1 22760F53
 P 2300 3700
@@
 $EndComp
 $Comp
-L CRYSTAL X3
+L video_schlib:CRYSTAL X3
 U 1 1 22760FA3
 P 2100 4800
