File: demos/video/video.kicad_pcb (KiCad board)
At the start: 4 copper layers, 312 x 106.7 mm, 189 parts, among them J4 DB9FEM, P1 BNC, P10 CONN_1, P11 CONN_1, P12 CONN_1, P2 BNC, P3 BNC, P4 CONN_2, P5 CONN_5, P8 BNC, P9 CONN_1, Q1 BC848, Q2 BC848, Q3 BC848, U1 24C16, U10 BT812, U11 S5933_PQ160, U12 SIM4X32, U13 SIM4X32, U14 SIM4X32, U15 SIM4X32, U16 SIM4X32, U17 SIM4X32, U18 SIM4X32, U19 SIM4X32, U2 4C4001, U20 TDA8501, U21 XC1736APD8, U22 XC4003-VQ100, U23 XC4003/PQ100, U24 XC4005-PQ160, U3 74LS245, U4 74LS245, U5 74LS245, U6 74LS245, U7 AV9173, U8 BT253, U9 BT473, X1 10MHz, X2 30MHz, X3 4.433618MHz

Commit message: New upstream version 5.0.0~rc3+dfsg1
Parts:
- moved R35 1.75 mm to (353.5, 59.3), turned to 90 degrees
- moved RR6 0.29 mm to (84.8, 127.0)
- moved C37 0.25 mm to (318.9, 120.0)
Connections:
- U10 pad 101: (no net) -> Net-(U10-Pad101)
- U10 pad 105: (no net) -> Net-(U10-Pad105)
- U10 pad 106: (no net) -> Net-(U10-Pad106)
- U10 pad 107: (no net) -> Net-(U10-Pad107)
- U10 pad 127: (no net) -> Net-(U10-Pad127)
- U10 pad 129: (no net) -> Net-(U10-Pad129)
- U10 pad 131: (no net) -> Net-(U10-Pad131)
- U10 pad 150: (no net) -> Net-(U10-Pad150)
- U10 pad 152: (no net) -> Net-(U10-Pad152)
- U10 pad 154: (no net) -> Net-(U10-Pad154)
- U10 pad 25: (no net) -> Net-(U10-Pad25)
- U10 pad 26: (no net) -> Net-(U10-Pad26)
- U10 pad 27: (no net) -> Net-(U10-Pad27)
- U10 pad 28: (no net) -> Net-(U10-Pad28)
- U10 pad 29: (no net) -> Net-(U10-Pad29)
- U10 pad 32: (no net) -> Net-(U10-Pad32)
- U10 pad 33: (no net) -> Net-(U10-Pad33)
- U10 pad 35: (no net) -> Net-(U10-Pad35)
- U10 pad 37: (no net) -> Net-(U10-Pad37)
- U10 pad 38: (no net) -> Net-(U10-Pad38)
- U12 pad 67: (no net) -> Net-(U12-Pad67)
- U12 pad 68: (no net) -> Net-(U12-Pad68)
- U12 pad 69: (no net) -> Net-(U12-Pad69)
- U12 pad 70: (no net) -> Net-(U12-Pad70)
- U13 pad 67: (no net) -> Net-(U13-Pad67)
- U13 pad 68: (no net) -> Net-(U13-Pad68)
- U13 pad 69: (no net) -> Net-(U13-Pad69)
- U13 pad 70: (no net) -> Net-(U13-Pad70)
- U14 pad 67: (no net) -> Net-(U14-Pad67)
- U14 pad 68: (no net) -> Net-(U14-Pad68)
- U14 pad 69: (no net) -> Net-(U14-Pad69)
- U14 pad 70: (no net) -> Net-(U14-Pad70)
- U15 pad 67: (no net) -> Net-(U15-Pad67)
- U15 pad 68: (no net) -> Net-(U15-Pad68)
- U15 pad 69: (no net) -> Net-(U15-Pad69)
- U15 pad 70: (no net) -> Net-(U15-Pad70)
- U16 pad 67: (no net) -> Net-(U16-Pad67)
- U16 pad 68: (no net) -> Net-(U16-Pad68)
- U16 pad 69: (no net) -> Net-(U16-Pad69)
- U16 pad 70: (no net) -> Net-(U16-Pad70)
- U17 pad 67: (no net) -> Net-(U17-Pad67)
- U17 pad 68: (no net) -> Net-(U17-Pad68)
- U17 pad 69: (no net) -> Net-(U17-Pad69)
- U17 pad 70: (no net) -> Net-(U17-Pad70)
- U18 pad 67: (no net) -> Net-(U18-Pad67)
- U18 pad 68: (no net) -> Net-(U18-Pad68)
- U18 pad 69: (no net) -> Net-(U18-Pad69)
- U18 pad 70: (no net) -> Net-(U18-Pad70)
- U19 pad 67: (no net) -> Net-(U19-Pad67)
- U19 pad 68: (no net) -> Net-(U19-Pad68)
- U19 pad 69: (no net) -> Net-(U19-Pad69)
- U19 pad 70: (no net) -> Net-(U19-Pad70)
- U20 pad 1: (no net) -> Net-(U20-Pad1)
- U20 pad 3: (no net) -> Net-(U20-Pad3)
- U20 pad 4: (no net) -> Net-(U20-Pad4)
- U20 pad 5: (no net) -> Net-(U20-Pad5)
- U21 pad 6: (no net) -> Net-(U21-Pad6)
- U22 pad 10: (no net) -> Net-(U22-Pad10)
- U22 pad 14: (no net) -> Net-(U22-Pad14)
- U22 pad 15: (no net) -> Net-(U22-Pad15)
- U22 pad 16: (no net) -> Net-(U22-Pad16)
- U22 pad 27: (no net) -> Net-(U22-Pad27)
- U22 pad 3: (no net) -> Net-(U22-Pad3)
- U22 pad 30: (no net) -> Net-(U22-Pad30)
- U22 pad 4: (no net) -> Net-(U22-Pad4)
- U22 pad 5: (no net) -> Net-(U22-Pad5)
- U22 pad 6: (no net) -> Net-(U22-Pad6)
- U22 pad 65: (no net) -> Net-(U22-Pad65)
- U22 pad 66: (no net) -> Net-(U22-Pad66)
- U22 pad 73: (no net) -> Net-(U22-Pad73)
- U22 pad 76: (no net) -> Net-(U22-Pad76)
- U23 pad 100: (no net) -> Net-(U23-Pad100)
- U23 pad 2: (no net) -> Net-(U23-Pad2)
- U23 pad 31: (no net) -> Net-(U23-Pad31)
- U23 pad 33: (no net) -> Net-(U23-Pad33)
- U23 pad 49: (no net) -> Net-(U23-Pad49)
- U23 pad 50: (no net) -> Net-(U23-Pad50)
- U23 pad 58: (no net) -> Net-(U23-Pad58)
- U23 pad 60: (no net) -> Net-(U23-Pad60)
- U23 pad 62: (no net) -> Net-(U23-Pad62)
- U23 pad 68: (no net) -> Net-(U23-Pad68)
- U23 pad 76: (no net) -> Net-(U23-Pad76)
- U23 pad 79: (no net) -> Net-(U23-Pad79)
- U23 pad 98: (no net) -> Net-(U23-Pad98)
- U23 pad 99: (no net) -> Net-(U23-Pad99)
- U24 pad 121: (no net) -> Net-(U24-Pad121)
- U24 pad 84: (no net) -> Net-(U24-Pad84)
- U7 pad 8: (no net) -> Net-(U7-Pad8)
- U8 pad 4: (no net) -> Net-(U8-Pad4)
- U8 pad 5: (no net) -> Net-(U8-Pad5)
- U8 pad 74: (no net) -> Net-(U8-Pad74)
- U8 pad 77: (no net) -> Net-(U8-Pad77)
- U8 pad 81: (no net) -> Net-(U8-Pad81)
- U9 pad 27: (no net) -> Net-(U9-Pad27)
- U9 pad 30: (no net) -> Net-(U9-Pad30)
- U9 pad 5: (no net) -> Net-(U9-Pad5)
- U9 pad 6: (no net) -> Net-(U9-Pad6)
Routing:
- net /PTRDY-: track 109.7 -> 111.0 mm
- net /muxdata/DPC19: track 73.0 -> 74.0 mm
- net /muxdata/DPC20: track 94.8 -> 95.7 mm
- net /muxdata/DPC18: track 77.6 -> 78.5 mm
- net /buspci.sch/EA12: track 39.8 -> 40.7 mm
- net /buspci.sch/EA11: track 35.1 -> 36.1 mm
- net /buspci.sch/EA13: track 34.4 -> 35.4 mm
- net Net-(C1-Pad1): track 5.08 -> 5.99 mm
- net /pal-ntsc.sch/Y_SYNC: track 13.4 -> 12.6 mm
- net /buspci.sch/EA10: track 32.8 -> 33.6 mm
