File: kicad/demos/interf_u/interf_u.sch (KiCad schematic (older format))
At the start: 24 parts, among them P1 DB25FEMELLE, U1 74LS245, U2 74LS688, U3 74LS541, U5 628128, U8 EP600, U9 4003APG120, X1 8MHz

Commit message: Imported Upstream version 0.0.20110507
Parts:
- U9: Field5 (none) -> test; price (none) -> 50$
Connections:
- wire segments 312 -> 278
Changed lines of the file:
@@
-EESchema Schematic File Version 2  date 28/04/2010 09:06:34
+EESchema Schematic File Version 2  date 02/02/2011 07:13:59
 LIBS:power
 LIBS:device
@@
 LIBS:special
 LIBS:interf_u-cache
-EELAYER 24  0
+EELAYER 25  0
 EELAYER END
 $Descr A3 16535 11700
 Sheet 1 1
 Title "INTERFACE UNIVERSEL"
-Date "28 apr 2010"
+Date "7 dec 2010"
 Rev "2B"
 Comp "KICAD"
@@
 	3150 2250 3650 2250
 Wire Wire Line
-	4450 9300 3800 9300
-Wire Wire Line
-	3800 9300 3250 9300
-Wire Wire Line
-	3250 9300 2600 9300
+	4450 9300 2600 9300
 Wire Wire Line
 	2600 9300 2600 9350
@@
 	2600 8900 2600 8850
 Wire Wire Line
-	4450 8900 3800 8900
-Wire Wire Line
-	3800 8900 3250 8900
-Wire Wire Line
-	3250 8900 2600 8900
+	4450 8900 2600 8900
 Connection ~ 3250 8900
 Connection ~ 3800 8900
@@
 	10050 3300 10100 3300
 Wire Wire Line
-	10050 3000 10050 3100
-Wire Wire Line
-	10050 3100 10050 3200
-Wire Wire Line
-	10050 3200 10050 3300
+	10050 3000 10050 3300
 Wire Wire Line
 	10100 3100 10050 3100
@@
 Connection ~ 10050 3200
 Wire Wire Line
-	13550 4400 13550 4150
-Wire Wire Line
-	13550 4150 13550 3700
-Wire Wire Line
-	14350 4400 14350 4150
-Wire Wire Line
-	14350 4150 14350 3700
+	13550 4400 13550 3700
+Wire Wire Line
+	14350 4400 14350 3700
 Connection ~ 13550 4150
 Connection ~ 14350 4150
@@
 	8450 1850 9000 1850
 Wire Wire Line
-	8450 1950 8500 1950
-Wire Wire Line
-	8500 1950 9000 1950
+	8450 1950 9000 1950
 Wire Wire Line
 	8450 2150 9000 2150
@@
 	3950 4000 4500 4000
 Wire Wire Line
-	4550 2350 4550 2450
-Wire Wire Line
-	4550 2450 4550 2550
+	4550 2350 4550 2550
 Connection ~ 4550 2450
 Wire Wire Line
@@
 	14700 7500 14750 7500
 Wire Wire Line
-	14700 7500 14700 7300
-Wire Wire Line
-	14700 7300 14700 7100
-Wire Wire Line
-	14700 7100 14700 6900
-Wire Wire Line
-	14700 6900 14700 6700
-Wire Wire Line
-	14700 6700 14700 6500
-Wire Wire Line
-	14700 6500 14700 6300
-Wire Wire Line
-	14700 6300 14700 6100
-Wire Wire Line
-	14650 6100 14700 6100
-Wire Wire Line
-	14700 6100 14750 6100
+	14700 7500 14700 6100
+Wire Wire Line
+	14650 6100 14750 6100
 Wire Wire Line
 	14750 6300 14700 6300
@@
 	1200 6900 1300 6900
 Wire Wire Line
-	1200 7700 1200 7600
-Wire Wire Line
-	1200 7600 1200 7500
-Wire Wire Line
-	1200 7500 1200 7400
-Wire Wire Line
-	1200 7400 1200 7300
-Wire Wire Line
-	1200 7300 1200 7200
-Wire Wire Line
-	1200 7200 1200 7100
-Wire Wire Line
-	1200 7100 1200 7000
-Wire Wire Line
-	1200 7000 1200 6900
+	1200 7700 1200 6900
 Wire Wire Line
 	1300 7000 1200 7000
@@
 	3350 6800 3350 6900
 Wire Wire Line
-	3350 6800 3150 6800
-Wire Wire Line
-	3150 6800 2450 6800
+	3350 6800 2450 6800
 Wire Wire Line
 	2450 6800 2450 6900
@@
 	3150 7950 3150 6800
 Wire Wire Line
-	3900 7000 2950 7000
-Wire Wire Line
-	2950 7000 2600 7000
+	3900 7000 2600 7000
 Wire Wire Line
 	2600 7000 2600 7100
@@
 	3050 6900 2500 6900
 Wire Wire Line
-	3050 7950 3050 7700
-Wire Wire Line
-	3050 7700 3050 6900
+	3050 7950 3050 6900
 Wire Wire Line
 	3900 7600 3400 7600
@@
 	3400 7700 3050 7700
 Wire Wire Line
-	2100 7300 2750 7300
-Wire Wire Line
-	2750 7300 3250 7300
+	2100 7300 3250 7300
 Wire Wire Line
 	3250 7300 3250 7100
@@
 	3250 7100 3900 7100
 Wire Wire Line
-	2100 7600 2450 7600
-Wire Wire Line
-	2450 7600 3300 7600
+	2100 7600 3300 7600
 Wire Wire Line
 	3300 7600 3300 7300
@@
 	3900 7500 2850 7500
 Wire Wire Line
-	3900 7400 2650 7400
-Wire Wire Line
-	2650 7400 2100 7400
+	3900 7400 2100 7400
 Connection ~ 2450 7600
 Connection ~ 2550 7500
@@
 	2850 7200 2100 7200
 Wire Wire Line
-	2850 7950 2850 7500
-Wire Wire Line
-	2850 7500 2850 7200
-Wire Wire Line
-	2550 7950 2550 7500
-Wire Wire Line
-	2550 7500 2550 7150
+	2850 7950 2850 7200
+Wire Wire Line
+	2550 7950 2550 7150
 Wire Wire Line
 	2550 7150 2900 7150
@@
 	14250 4150 14350 4150
 Wire Bus Line
-	3750 2350 3750 2250
+	3750 2350 3750 1650
 Wire Bus Line
-	3750 2250 3750 2150
-Wire Bus Line
-	3750 2150 3750 2050
-Wire Bus Line
-	3750 2050 3750 1950
-Wire Bus Line
-	3750 1950 3750 1850
-Wire Bus Line
-	3750 1850 3750 1750
-Wire Bus Line
-	3750 1750 3750 1650
-Wire Bus Line
-	3750 3450 3750 3550
-Wire Bus Line
-	3750 3550 3750 3650
-Wire Bus Line
-	3750 3650 3750 3750
-Wire Bus Line
-	3750 3750 3750 3850
-Wire Bus Line
-	3750 3850 3750 3950
-Wire Bus Line
-	3750 3950 3750 4050
-Wire Bus Line
-	3750 4050 3750 4150
-Wire Bus Line
-	3750 4150 3750 4250
-Wire Bus Line
-	3750 4250 3750 4350
-Wire Bus Line
-	3750 4350 3750 4450
-Wire Bus Line
-	3750 4450 3750 4550
-Wire Bus Line
-	3750 4550 3750 5350
+	3750 3450 3750 5350
 Wire Bus Line
 	3300 5350 3750 5350
 Wire Bus Line
-	3300 6650 3300 6550
+	3300 6650 3300 5350
 Wire Bus Line
-	3300 6550 3300 6450
-Wire Bus Line
-	3300 6450 3300 6350
-Wire Bus Line
-	3300 6350 3300 6250
-Wire Bus Line
-	3300 6250 3300 6150
-Wire Bus Line
-	3300 6150 3300 6050
-Wire Bus Line
-	3300 6050 3300 5950
-Wire Bus Line
-	3300 5950 3300 5350
-Wire Bus Line
-	3900 3700 3900 3600
-Wire Bus Line
-	3900 3600 3900 3500
-Wire Bus Line
-	3900 3500 3900 3400
-Wire Bus Line
-	3900 3400 3900 3300
-Wire Bus Line
-	3900 3300 3900 3200
-Wire Bus Line
-	3900 3200 3900 3100
-Wire Bus Line
-	3900 3100 3900 3000
-Wire Bus Line
-	3900 3000 3900 2450
-Wire Wire Line
-	13700 3700 13550 3700
-Wire Wire Line
-	13550 3700 12300 3700
-Wire Wire Line
-	14200 3700 14350 3700
-Wire Wire Line
-	14350 3700 14650 3700
+	3900 3700 3900 2450
+Wire Wire Line
+	13700 3700 12300 3700
+Wire Wire Line
+	14200 3700 14650 3700
 Wire Wire Line
 	15200 3700 15150 3700
@@
 Text Label 9700 4600 0    60   ~ 0
 MA15
-Text Label 13050 1050 0    60   ~ 0
+Text Label 13000 1050 0    60   ~ 0
 LED1
-Text Label 13050 1500 0    60   ~ 0
+Text Label 13000 1500 0    60   ~ 0
 LED2
 Text Label 9700 4200 0    60   ~ 0
@@
 F 1 "4003APG120" H 11200 2950 70  0000 C CNN
 F 2 "PGA120" H 11200 2850 60  0000 C CNN
+F 4 "50$" H 11200 5700 60  0001 C CNN "price"
+F 5 "test" H 11200 5700 60  0001 C CNN "Field5"
 	1    11200 5700
 	1    0    0    -1
