File: kicad/demos/pspice/pspice.sch (KiCad schematic (older format))
At the start: 20 parts, among them Q1 Q2N2222, Q2 Q2N2222, Q3 Q2N2222

Commit message: Imported Upstream version 0.0.20110507
Other:
- note added: "+gnucap .model Q2N2222 npn (bf=200)\n.print tran v(nodes)\n.print dc v(nodes)\n.tran 10 10000 10 > pspice.dat\n"
- note added: "Pspice directives using one multiline text:"
- note removed: "+PSPICE .print ac v(vout)"
- note removed: "+gnucap .plot ac v(nodes) (-1,5)"
- note removed: "-PSPICE .DC V1 10 12 0.5"
- note removed: "-PSPICE .model Q2N2222 npn (bf=200)"
- note removed: "-gnucap .AC 10 1Meg *1.2"
