File: demos/complex_hierarchy/ampli_ht.sch (KiCad schematic (older format))
At the start: 29 parts, among them P5 CONN_2, P6 CONN_2, Q5 MPAS92, Q6 MPAS42, Q7 MPAS92, Q8 MPAS42, U4 LM358N

Commit message: Imported Upstream version 4.0.0~rc1
Parts:
- C12, C6, C8: footprint (none) -> discret:C2
- C7: value 4,7nF -> 4.7nF; footprint (none) -> discret:C2
- D5, D6, D7, D8: footprint (none) -> discret:D3; symbol DIODE -> D_Small
- P5, P6: footprint (none) -> connect:bornier2
- Q5, Q6, Q7, Q8: footprint (none) -> discret:TO92-CBE
- R10, R13, R14, R15, R16, R17, R18, R19, R21, R22, R23, R25, R26: footprint (none) -> discret:R3-LARGE_PADS
- RV2: footprint (none) -> discret:RV2
- U4: footprint (none) -> dip_sockets:DIP-8__300_ELL
Connections:
- wire segments 56 -> 68
Other:
- note added: "Filter:\nFc =1000Hz"
- note removed: "Filtre:\nFc =1000Hz"
- moved on the sheet: U4A, U4B
