File: demos/complex_hierarchy/complex_hierarchy.sch (KiCad schematic (older format))
At the start: 10 parts, among them P1 CONN_2, P2 CONN_2, U1 ICL7660, U2 78L05

Commit message: New upstream version 5.0.0~rc1+dfsg1
Parts:
- C1, C10, C11, C2, C9: symbol CP -> complex_hierarchy_schlib:CP
- D1: footprint Discret:D5 -> Diode_THT:D_DO-41_SOD81_P12.70mm_Horizontal; symbol D_Small -> complex_hierarchy_schlib:D_Small
- P1, P2: footprint Connect:bornier2 -> TerminalBlock_Phoenix:TerminalBlock_Phoenix_MKDS-1,5-2-5.08_1x02_P5.08mm_Horizontal; symbol CONN_2 -> complex_hierarchy_schlib:CONN_2
- U1: footprint dip_sockets:DIP-8__300_ELL -> Package_DIP:DIP-8_W7.62mm_LongPads; symbol ICL7660 -> complex_hierarchy_schlib:ICL7660
- U2: symbol 7805 -> complex_hierarchy_schlib:7805
Connections:
- wire segments 38 -> 46
Changed lines of the file:
@@
-EESchema Schematic File Version 2
-LIBS:power
-LIBS:complex_hierarchy_schlib
+EESchema Schematic File Version 4
 LIBS:complex_hierarchy-cache
-EELAYER 25 0
+EELAYER 26 0
 EELAYER END
 $Descr A4 11693 8268
 encoding utf-8
 Sheet 1 3
-Title ""
-Date "21 mar 2015"
+Title "Complex hierarchy: demo"
+Date "2017-01-15"
 Rev ""
 Comp ""
@@
 	8300 1300 9200 1300
 Wire Wire Line
-	2800 2500 3800 2500
-Wire Wire Line
-	2500 1250 2500 1350
+	2800 2500 3000 2500
+Wire Wire Line
+	2500 1250 2500 1300
 Wire Wire Line
 	3800 2500 3800 2450
@@
 	9200 1750 9200 1800
 Wire Wire Line
-	9200 1250 9200 1450
+	9200 1250 9200 1300
 Connection ~ 9200 1300
 Wire Wire Line
-	2200 1650 2200 1750
+	2200 1650 2200 1700
 Wire Wire Line
 	2500 1650 2500 1700
@@
 	7050 2650 7100 2650
 Wire Wire Line
-	8800 2750 9350 2750
-$Comp
-L CP C10
+	8800 2750 9200 2750
+$Comp
+L complex_hierarchy_schlib:CP C10
 U 1 1 4B4B15E7
 P 6650 2750
 F 0 "C10" H 6800 2800 50  0000 L CNN
 F 1 "10uF" H 6800 2750 50  0000 L TNN
-F 2 "Discret:CP6" H 6650 2750 60  0001 C CNN
+F 2 "Discret:CP6" H 6850 2650 30  0000 C CNN
 F 3 "" H 6650 2750 60  0001 C CNN
 	1    6650 2750
@@
 $EndComp
 $Comp
-L GND #PWR01
+L complex_hierarchy_schlib:GND #PWR01
 U 1 1 4B4B15DA
 P 9050 2300
@@
 $EndComp
 $Comp
-L CP C11
+L complex_hierarchy_schlib:CP C11
 U 1 1 4B4B15D9
 P 9200 2500
 F 0 "C11" H 9350 2550 50  0000 L CNN
 F 1 "10uF" H 9350 2500 50  0000 L TNN
-F 2 "Discret:CP6" H 9200 2500 60  0001 C CNN
+F 2 "Discret:CP6" H 9550 2400 30  0000 C CNN
 F 3 "" H 9200 2500 60  0001 C CNN
 	1    9200 2500
@@
 NoConn ~ 7100 3050
 $Comp
-L -VAA #PWR02
+L complex_hierarchy_schlib:-VAA #PWR02
 U 1 1 4B4B1578
 P 9350 2750
@@
 $EndComp
 $Comp
-L 7805 U2
+L complex_hierarchy_schlib:7805 U2
 U 1 1 4B4B1532
 P 7900 1350
 F 0 "U2" H 7900 1650 60  0000 C CNN
 F 1 "78L05" H 7900 1550 60  0000 C CNN
-F 2 "Discret:LM78LXX" H 7900 1350 60  0001 C CNN
+F 2 "Discret:LM78LXX" H 8100 1150 30  0000 C CNN
 F 3 "" H 7900 1350 60  0001 C CNN
 	1    7900 1350
@@
 $EndComp
 $Comp
-L VCC #PWR03
+L complex_hierarchy_schlib:VCC #PWR03
 U 1 1 4B4B1253
 P 7900 2200
@@
 $EndComp
 $Comp
-L VCC #PWR04
+L complex_hierarchy_schlib:VCC #PWR04
 U 1 1 4B4B124E
 P 9200 1250
@@
 $EndComp
 $Comp
-L GND #PWR05
+L complex_hierarchy_schlib:GND #PWR05
 U 1 1 4B4B1237
 P 7900 3600
@@
 $EndComp
 $Comp
-L ICL7660 U1
+L complex_hierarchy_schlib:ICL7660 U1
 U 1 1 4B4B1230
 P 7950 2900
 F 0 "U1" H 7400 3300 70  0000 L CNN
 F 1 "ICL7660" H 8500 2450 70  0000 R CNN
-F 2 "dip_sockets:DIP-8__300_ELL" H 7950 2900 60  0001 C CNN
+F 2 "Package_DIP:DIP-8_W7.62mm_LongPads" H 8950 2300 60  0000 C CNN
 F 3 "" H 7950 2900 60  0001 C CNN
 	1    7950 2900
@@
 12Vext
 $Comp
-L CP C9
+L complex_hierarchy_schlib:CP C9
 U 1 1 4B3A1558
 P 2500 1500
 F 0 "C9" H 2650 1550 50  0000 L CNN
 F 1 "47uF/63V" H 2650 1500 50  0000 L TNN
-F 2 "Discret:CP8" H 2500 1500 60  0001 C CNN
+F 2 "Discret:CP8" H 2800 1400 30  0000 C CNN
 F 3 "" H 2500 1500 60  0001 C CNN
 	1    2500 1500
@@
 $EndComp
 $Comp
-L GND #PWR06
+L complex_hierarchy_schlib:GND #PWR06
 U 1 1 4B3A1557
 P 2500 1700
@@
 $EndSheet
 $Comp
-L GND #PWR07
+L complex_hierarchy_schlib:GND #PWR07
 U 1 1 4B3A1302
 P 2200 1750
@@
 $EndComp
 $Comp
-L CONN_2 P1
+L complex_hierarchy_schlib:CONN_2 P1
 U 1 1 4B3A12F4
 P 1650 1400
 F 0 "P1" V 1600 1400 40  0000 C CNN
 F 1 "CONN_2" V 1700 1400 40  0000 C CNN
-F 2 "Connect:bornier2" H 1650 1400 60  0001 C CNN
+F 2 "TerminalBlock_Phoenix:TerminalBlock_Phoenix_MKDS-1,5-2-5.08_1x02_P5.08mm_Horizontal" H 1650 1200 30  0000 C CNN
 F 3 "" H 1650 1400 60  0001 C CNN
 	1    1650 1400
@@
 $EndComp
 $Comp
-L HT #PWR08
+L complex_hierarchy_schlib:HT #PWR08
 U 1 1 4B0FA68B
 P 2500 1250
@@
 $EndComp
 $Comp
-L CP C1
+L complex_hierarchy_schlib:CP C1
 U 1 1 4B03CEC2
 P 9200 1600
 F 0 "C1" H 9350 1650 50  0000 L CNN
 F 1 "47uF" H 9350 1600 50  0000 L TNN
-F 2 "Discret:CP6" H 9200 1600 60  0001 C CNN
+F 2 "Discret:CP6" H 9500 1500 30  0000 C CNN
 F 3 "" H 9200 1600 60  0001 C CNN
 	1    9200 1600
@@
 $EndComp
 $Comp
-L GND #PWR09
+L complex_hierarchy_schlib:GND #PWR09
 U 1 1 4B03CEC1
 P 9200 1800
@@
 $EndComp
 $Comp
-L GND #PWR010
+L complex_hierarchy_schlib:GND #PWR010
 U 1 1 4B03CE88
 P 7900 1650
@@
 $EndComp
 $Comp
-L +12C #PWR011
+L complex_hierarchy_schlib:+12C #PWR011
 U 1 1 4B03CE6C
 P 7400 1250
@@
 $EndComp
 $Comp
-L PWR_FLAG #U012
+L complex_hierarchy_schlib:PWR_FLAG #U012
 U 1 1 4B03CAA3
 P 2200 1250
@@
 $EndComp
 $Comp
-L PWR_FLAG #U013
+L complex_hierarchy_schlib:PWR_FLAG #U013
 U 1 1 4B03C9F9
 P 3000 2450
@@
 $EndComp
 $Comp
-L +12C #PWR014
+L complex_hierarchy_schlib:+12C #PWR014
 U 1 1 4B03C68D
 P 3800 2450
@@
 $EndComp
 $Comp
-L PWR_FLAG #U015
+L complex_hierarchy_schlib:PWR_FLAG #U015
 U 1 1 4AE17C31
 P 2200 1650
@@
 $EndComp
 $Comp
-L +12V #U016
+L complex_hierarchy_schlib:+12V #U016
 U 1 1 4AE173EF
 P 3550 2450
@@
 $EndComp
 $Comp
-L GND #PWR017
+L complex_hierarchy_schlib:GND #PWR017
 U 1 1 4AE173D0
 P 3200 3000
@@
 $EndComp
 $Comp
-L CP C2
+L complex_hierarchy_schlib:CP C2
 U 1 1 4AE173CF
 P 3200 2750
 F 0 "C2" H 3350 2800 50  0000 L CNN
 F 1 "47uF/20V" H 3350 2700 50  0000 L TNN
-F 2 "Discret:CP6" H 3200 2750 60  0001 C CNN
+F 2 "Discret:CP6" H 3550 2600 30  0000 C CNN
 F 3 "" H 3200 2750 60  0001 C CNN
 	1    3200 2750
@@
 $EndComp
 $Comp
-L D_Small D1
+L complex_hierarchy_schlib:D_Small D1
 U 1 1 4AE172F4
 P 2700 2500
 F 0 "D1" H 2700 2400 40  0000 C CNN
 F 1 "1N4007" H 2700 2600 40  0000 C CNN
-F 2 "Discret:D5" H 2700 2500 60  0001 C CNN
+F 2 "Diode_THT:D_DO-41_SOD81_P12.70mm_Horizontal" H 2700 2350 30  0000 C CNN
 F 3 "" H 2700 2500 60  0001 C CNN
 	1    2700 2500
@@
 $EndComp
 $Comp
-L GND #PWR018
+L complex_hierarchy_schlib:GND #PWR018
 U 1 1 4AD71B8E
 P 2100 2800
@@
 $EndComp
 $Comp
-L CONN_2 P2
+L complex_hierarchy_schlib:CONN_2 P2
 U 1 1 4AD71B06
 P 1650 2600
 F 0 "P2" V 1600 2600 40  0000 C CNN
 F 1 "CONN_2" V 1700 2600 40  0000 C CNN
-F 2 "Connect:bornier2" H 1650 2600 60  0001 C CNN
+F 2 "TerminalBlock_Phoenix:TerminalBlock_Phoenix_MKDS-1,5-2-5.08_1x02_P5.08mm_Horizontal" H 1650 2400 30  0000 C CNN
 F 3 "" H 1650 2600 60  0001 C CNN
 	1    1650 2600
@@
 Connection ~ 2200 1300
 Wire Wire Line
-	2000 1300 2500 1300
+	2000 1300 2200 1300
 Wire Wire Line
 	2000 1500 2100 1500
@@
 Wire Wire Line
 	7900 3600 7900 3550
+Wire Wire Line
+	9200 2750 9350 2750
+Wire Wire Line
+	2500 1300 2500 1350
+Wire Wire Line
+	3200 2500 3550 2500
+Wire Wire Line
+	3550 2500 3800 2500
+Wire Wire Line
+	3000 2500 3200 2500
+Wire Wire Line
+	9200 1300 9200 1450
+Wire Wire Line
+	2200 1300 2500 1300
+Wire Wire Line
+	2200 1700 2200 1750
 $EndSCHEMATC
