File: demos/ecc83/ecc83-pp.kicad_pcb (KiCad board)
At the start: 2 copper layers, 44.5 x 41.9 mm, 15 parts, among them P1 IN, P2 OUT, P3 POWER, P4 CONN_2, P5 CONN_1, P6 CONN_1, P7 CONN_1, P8 CONN_1, U1 ECC83

Commit message: New upstream version 5.0.0~rc1+dfsg1
Parts:
- P1, P2, P3, P4: footprint connect:bornier2 -> TerminalBlock_Phoenix:TerminalBlock_Phoenix_MKDS-1,5-2_1x02_P5.00mm_Horizontal
- U1: footprint Valves:VALVE-ECC-83-1 -> Valve:Valve_ECC-83-1
- moved P1 5.21 mm to (164.6, 105.3), turned to 90 degrees
- moved P7 4.19 mm to (165.1, 133.7)
- moved P8 4.19 mm to (127.0, 133.7)
- moved R3 4.14 mm to (130.0, 123.8), turned to 180 degrees
- moved P2 4.06 mm to (128.3, 112.8), turned to 270 degrees
- moved P4 2.92 mm to (145.5, 131.2), turned to 0 degrees
- moved P3 2.16 mm to (128.3, 100.7), turned to 270 degrees
- moved C1 1.53 mm to (139.4, 97.3)
- moved R2 1.40 mm to (151.3, 97.8)
Connections:
- U1 pad 4: Net-(P4-Pad1) -> Net-(P4-Pad2)
- U1 pad 5: Net-(P4-Pad1) -> Net-(P4-Pad2)
- U1 pad 9: Net-(P4-Pad2) -> Net-(P4-Pad1)
Routing:
- net Net-(P4-Pad2): track 11.3 -> 27.9 mm
- net Net-(P4-Pad1): track 26.2 -> 11.3 mm
- net Net-(P1-Pad2): track 14.9 -> 29.1 mm
- net Net-(C2-Pad1): track 12.5 -> 19.1 mm
- net Net-(R1-Pad1): track 64.8 -> 68.6 mm
- net Net-(R2-Pad1): track 20.5 -> 19.1 mm
- net GND: track 12.3 -> 11.2 mm
- net Net-(C1-Pad1): track 25.6 -> 24.6 mm
Other:
- board size 44.5 x 41.9 mm -> 44.5 x 45.7 mm
