File: demos/ecc83/ecc83-pp_v2.kicad_pcb (KiCad board)
At the start: 2 copper layers, 15 parts, among them P1 IN, P2 OUT, P3 POWER, P4 CONN_2, U1 ECC83

Commit message: Imported Upstream version 4.0.0~rc1
Parts:
- removed 1PIN (x3): P***, 1pin
- removed 1PIN: GND, 1pin
- added P5: CONN_1, connect:1pin, F.Cu at (123.2, 94.0)
- added P6: CONN_1, connect:1pin, F.Cu at (165.1, 94.0)
- added P7: CONN_1, connect:1pin, F.Cu at (165.1, 129.5)
- added P8: CONN_1, connect:1pin, F.Cu at (123.2, 129.5)
- C1: footprint C2V10 -> discret:C2V10
- C2: footprint CP8 -> discret:CP8
- P1, P2, P3, P4: footprint PIN_ARRAY_2X1 -> pin_array:pin_array_1x02
- R1, R2, R3, R4: footprint R3 -> discret:R3
- U1: footprint ECC-83-2 -> Valves:VALVE-ECC-83-2
- moved U1 0.08 mm to (149.3, 109.2)
Routing:
- net GND: track 99.9 -> 0.25 mm
Other:
- board outline added: 48.3 x 41.9 mm
- rule pad_to_mask_clearance: 0.254 -> 0.1
- rule trace_min: 0.254 -> 0.154
