File: demos/flat_hierarchy/pic_programmer.sch (KiCad schematic (older format))
At the start: 50 parts, among them J1 DB9-FEMAL, P1 CONN_2, Q1 BC237, Q2 BC307, Q3 BC307, U2 74HC125, U3 7805, U4 LT1373

Commit message: Imported Upstream version 4.0.0~rc1
Parts:
- D12: Champ4 (none) -> YELLOW-LED
- D8: Champ4 (none) -> Low Current Led; Champ5 (none) -> RED LED
- D9: Champ4 (none) -> GREEN LED
- R10: value 5,1K -> 5.1K
Connections:
- net labels added: VPP-MCLR
- net labels removed: VPP/MCLR
- wire segments 95 -> 119
Other:
- moved on the sheet: U4
