File: demos/flat_hierarchy/pic_programmer.sch (KiCad schematic (older format))
At the start: 50 parts, among them J1 DB9-FEMAL, P1 CONN_2, Q1 BC237, Q2 BC307, Q3 BC307, U2 74HC125, U3 7805, U4 LT1373

Commit message: New upstream version 5.0.0~rc1+dfsg1
Parts:
- C1, C2: footprint Discret:CP10 -> discret:CP10; symbol CP -> flat_hierarchy_schlib:CP
- C3: footprint Discret:CP8 -> discret:CP8; symbol CP -> flat_hierarchy_schlib:CP
- C4, C5, C9: footprint Discret:C1-1 -> discret:C1-1; symbol C -> flat_hierarchy_schlib:C
- D1: footprint Discret:D5 -> Diode_THT:D_DO-35_SOD27_P12.70mm_Horizontal; symbol DIODE -> device:D_ALT
- D10: footprint Discret:D5 -> Diode_THT:D_DO-35_SOD27_P12.70mm_Horizontal; symbol DIODESCH -> device:D_Schottky_ALT
- D11, D2, D3, D4, D5, D6, D7: footprint Discret:D3 -> Diode_THT:D_DO-35_SOD27_P7.62mm_Horizontal; symbol DIODESCH -> device:D_Schottky_ALT
- D12, D8, D9: footprint Discret:LEDV -> discret:LEDV; symbol LED -> flat_hierarchy_schlib:LED
- J1: footprint Connect:DB9FC -> connect:DB9FC; symbol DB9 -> flat_hierarchy_schlib:DB9
- JP1: symbol JUMPER -> flat_hierarchy_schlib:JUMPER
- L1: symbol INDUCTOR -> flat_hierarchy_schlib:INDUCTOR
- P1: footprint Connect:bornier2 -> connect:bornier2; symbol CONN_2 -> flat_hierarchy_schlib:CONN_2
- Q1: footprint Discret:TO92 -> discret:TO92; symbol NPN -> flat_hierarchy_schlib:NPN
- Q2, Q3: footprint Discret:TO92 -> discret:TO92; symbol PNP -> flat_hierarchy_schlib:PNP
- R1, R10, R11, R12, R13, R14, R15, R16, R17, R18, R19, R2, R20, R21, R3, R4, R5, R6, R7, R8, R9: footprint Discret:R4 -> Resistor_THT:R_Axial_DIN0207_L6.3mm_D2.5mm_P10.16mm_Horizontal; symbol R -> flat_hierarchy_schlib:R
- RV1: footprint Discret:RV2X4 -> discret:RV2X4; symbol POT -> flat_hierarchy_schlib:POT
- U2: footprint Sockets_DIP:DIP-10__300_ELL -> dip_sockets:DIP-14__300_ELL; symbol 74LS125 -> flat_hierarchy_schlib:74LS125
- U3: footprint Discret:LM78XX -> discret:LM78XX; symbol 7805 -> flat_hierarchy_schlib:7805
- U4: footprint Sockets_DIP:DIP-8__300_ELL -> dip_sockets:DIP-8__300_ELL; symbol LT1373 -> flat_hierarchy_schlib:LT1373
Connections:
- wire segments 119 -> 151
