File: demos/flat_hierarchy/pic_sockets.sch (KiCad schematic (older format))
At the start: 8 parts, among them P2 SUPP28, P3 SUPP40, U1 24Cxx, U5 PIC_18_PINS, U6 PIC_8_PINS

Commit message: Imported Upstream version 4.0.0~rc1
Connections:
- wire segments 28 -> 42
