File: demos/interf_u/interf_u.kicad_pcb (KiCad board)
At the start: 2 copper layers, 25 parts, among them P1 DB25FEMELLE, U1 74LS245, U2 74LS688, U3 74LS541, U5 628128, U8 EP600, U9 4003APG120, X1 8MHz

Commit message: Imported Upstream version 4.0.0~rc1
Parts:
- U1, U2, U3: footprint 20dip300 -> DIP-20__300
- U8: footprint 24dip300 -> DIP-24__300
- moved G1 136.5 mm to (25.9, 181.9)
Other:
- board outline added: 115.6 x 108 mm
