File: demos/interf_u/interf_u.sch (KiCad schematic (older format))
At the start: 24 parts, among them P1 DB25FEMELLE, U1 74LS245, U2 74LS688, U3 74LS541, U5 628128, U8 EP600, U9 4003APG120, X1 8MHz

Commit message: Imported Upstream version 4.0.0~rc1
Parts:
- C1, C4, C5, C6: footprint CP6 -> discret:CP6
- C2, C3: footprint C1 -> discret:C1
- D1, D2: footprint LEDV -> discret:LEDV
- P1: footprint DB25FC -> connect:DB25FC
- R1, R2, R3, R4, R5: footprint R3 -> discret:R3
- RR1: footprint r_pack9 -> discret:r_pack9
- U1, U2: footprint 20dip300 -> dip_sockets:DIP-20__300
- U3: footprint (none) -> dip_sockets:DIP-20__300
- U5: footprint 32dip600 -> dip_sockets:DIP-32__600
- U8: footprint 24dip300 -> dip_sockets:DIP-24__300
- X1: footprint HC-18UH -> discret:HC-18UH
Connections:
- wire segments 278 -> 294
Other:
- moved on the sheet: C1, C2, C3, C4, C5, C6

Commit message: New upstream version 5.0.0~rc1+dfsg1
Parts:
- BUS1: footprint BUS_PC -> interf_u:BUS_PC; symbol BUSPC -> interf_u_schlib:Bus_ISA_8bit
- C1, C4, C5, C6: footprint discret:CP6 -> Capacitor_THT:CP_Axial_L10.0mm_D4.5mm_P15.00mm_Horizontal; symbol CP -> interf_u_schlib:CP
- C2, C3: footprint discret:C1 -> Capacitor_THT:C_Disc_D3.0mm_W2.0mm_P2.50mm; symbol C -> interf_u_schlib:C
- D1, D2: footprint discret:LEDV -> LED_THT:LED_D5.0mm; symbol LED -> interf_u_schlib:LED
- JP1: footprint pin_array_8x2 -> Pin_Headers:Pin_Header_Straight_2x08; symbol CONN_8X2 -> interf_u_schlib:Conn_02x08_Odd_Even
- P1: footprint connect:DB25FC -> Connector_Dsub:DSUB-25_Female_Horizontal_P2.77x2.84mm_EdgePinOffset9.90mm_Housed_MountingHolesOffset11.32mm; symbol DB25 -> interf_u_schlib:DB25_Female
- R1, R2, R3, R4, R5: footprint discret:R3 -> Resistor_THT:R_Axial_DIN0207_L6.3mm_D2.5mm_P7.62mm_Horizontal; symbol R -> interf_u_schlib:R
- RR1: footprint discret:r_pack9 -> Resistor_THT:R_Array_SIP10; symbol RR9 -> interf_u_schlib:RR9
- U1: footprint dip_sockets:DIP-20__300 -> Package_DIP:DIP-20_W7.62mm; symbol 74LS245 -> interf_u_schlib:74LS245
- U2: footprint dip_sockets:DIP-20__300 -> Package_DIP:DIP-20_W7.62mm; symbol 74LS688 -> interf_u_schlib:74LS688
- U3: footprint dip_sockets:DIP-20__300 -> Package_DIP:DIP-20_W7.62mm; symbol 74LS541 -> interf_u_schlib:74LS541
- U5: footprint dip_sockets:DIP-32__600 -> Package_DIP:DIP-32_W15.24mm; symbol 628128 -> interf_u_schlib:628128
- U8: footprint dip_sockets:DIP-24__300 -> Package_DIP:DIP-24_W7.62mm; symbol EP600 -> interf_u_schlib:EP600
- U9: footprint PGA120 -> interf_u:PGA120; symbol 4003APG120 -> interf_u_schlib:4003APG120; Field5 test -> (none); price 50$ -> (none)
- X1: footprint discret:HC-18UH -> Crystal:Crystal_HC18-U_Horizontal; symbol CRYSTAL -> interf_u_schlib:Crystal
Connections:
- wire segments 294 -> 330
Other:
- moved on the sheet: C1, C2, C3, C4, C5, C6, D1, D2, R2, R3, R4, R5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
