File: demos/kit-dev-coldfire-xilinx_5213/kit-dev-coldfire-xilinx_5213.sch (KiCad schematic (older format))
At the start: 68 parts, among them Q1 3906, U1 MCF5213-LQFP100, U2 74AHC1G14, Y1 8MHz

Commit message: Imported Upstream version 4.0.0~rc1
Parts:
- ABRT_SW1, RST_SW1: footprint (none) -> discret:SW_PUSH_SMALL
- ALLPST1, CLKOUT1, GND1, TA-1: footprint (none) -> connect:PINTST
- BDM_EN1, CLK0, CLK1, CT1, VDDA1: footprint (none) -> pin_array:PIN_ARRAY_2X1
- BDM_PORT1: footprint (none) -> pin_array:pin_array_13x2
- C1, C10, C11, C12, C14, C15, C18, C2, C20, C21, C3, C4, C5, C6, C7, C8, C9, R1, R10, R11, R12, R13, R14, R15, R16, R17, R18, R19, R2, R20, R22, R25, R26, R4, R45, R46, R5, R6, R7, R8, R9: footprint (none) -> lib_smd:SM0805
- C16, C17, LEDABRT1, RED1: footprint (none) -> lib_smd:SM1206POL
- D1, D3: footprint (none) -> lib_smd:ST23AK#1
- FB1, L1, L2: footprint (none) -> lib_smd:SM1206
- LV1: footprint (none) -> discret:TO92-INVERT
- Q1: footprint (none) -> lib_smd:SOT23EBC
- R21: value 4,7K -> 4.7K; footprint (none) -> lib_smd:SM0805
- U1: footprint (none) -> lib_smd:VQFP100
- U2: footprint (none) -> lib_smd:SOT353
- Y1: footprint (none) -> discret:HC-18UH
Connections:
- wire segments 270 -> 373
Other:
- moved on the sheet: ABRT_SW1, ALLPST1, BDM_PORT1, C1, C10, C11, C12, C14, C15, C16, C17, C18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
