File: demos/kit-dev-coldfire-xilinx_5213/xilinx.sch (KiCad schematic (older format))
At the start: 21 parts, among them P1 CONN_6, P3 CONN_2X2, P4 CONN_20X2, U9 XCR3256-TQ144

Commit message: Imported Upstream version 4.0.0~rc1
Parts:
- C51, C52, C53, C54, C55, C56, C57, C58, C59, C60, C61, R57, R62, R63: footprint (none) -> lib_smd:SM0805
- D8, D9: footprint (none) -> lib_smd:SM1206POL
- P1: footprint (none) -> pin_array:PIN_ARRAY-6X1
- P3: footprint (none) -> pin_array:PIN_ARRAY_2X2
- P4: footprint (none) -> pin_array:PIN_ARRAY_20X2
- R64: footprint (none) -> discret:R4
- U9: footprint (none) -> lib_smd:TQFP144
Connections:
- wire segments 143 -> 172
Other:
- moved on the sheet: C51, C52, C53, C54, C55, C56, C57, C58, C59, C60, C61, D8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
