File: demos/kit-dev-coldfire-xilinx_5213/kit-dev-coldfire-xilinx_5213.kicad_pcb (KiCad board)
At the start: 4 copper layers, 157.5 x 91.4 mm, 162 parts, among them J1 JACK_2P, P1 CONN_6, P3 CONN_2X2, P4 CONN_20X2, Q1 3906, SW1 SW_PUSH, SW2 SW_PUSH, U1 MCF5213-LQFP100, U2 74AHC1G14, U3 MAX202, U4 74HC125, U5 MAX202, U7 PCA82C251, U8 MAX202, U9 XCR3256-TQ144, Y1 8MHz

Commit message: New upstream version 5.0.0~rc1+dfsg1
Connections:
- net VDD renamed +3.3V
- BDM_PORT1 pad 1: (no net) -> Net-(BDM_PORT1-Pad1)
- BDM_PORT1 pad 21: (no net) -> Net-(BDM_PORT1-Pad21)
- BDM_PORT1 pad 22: (no net) -> Net-(BDM_PORT1-Pad22)
- SW_ONOFF1 pad 1: (no net) -> Net-(SW_ONOFF1-Pad1)
- U9 pad 102: (no net) -> Net-(U9-Pad102)
- U9 pad 103: (no net) -> Net-(U9-Pad103)
- U9 pad 106: (no net) -> Net-(U9-Pad106)
- U9 pad 110: (no net) -> Net-(U9-Pad110)
- U9 pad 120: (no net) -> Net-(U9-Pad120)
- U9 pad 121: (no net) -> Net-(U9-Pad121)
- U9 pad 133: (no net) -> Net-(U9-Pad133)
- U9 pad 14: (no net) -> Net-(U9-Pad14)
- U9 pad 141: (no net) -> Net-(U9-Pad141)
- U9 pad 15: (no net) -> Net-(U9-Pad15)
- U9 pad 16: (no net) -> Net-(U9-Pad16)
- U9 pad 18: (no net) -> Net-(U9-Pad18)
- U9 pad 19: (no net) -> Net-(U9-Pad19)
- U9 pad 21: (no net) -> Net-(U9-Pad21)
- U9 pad 22: (no net) -> Net-(U9-Pad22)
- U9 pad 23: (no net) -> Net-(U9-Pad23)
- U9 pad 25: (no net) -> Net-(U9-Pad25)
- U9 pad 26: (no net) -> Net-(U9-Pad26)
- U9 pad 29: (no net) -> Net-(U9-Pad29)
- U9 pad 30: (no net) -> Net-(U9-Pad30)
- U9 pad 34: (no net) -> Net-(U9-Pad34)
- U9 pad 35: (no net) -> Net-(U9-Pad35)
- U9 pad 36: (no net) -> Net-(U9-Pad36)
- U9 pad 37: (no net) -> Net-(U9-Pad37)
- U9 pad 38: (no net) -> Net-(U9-Pad38)
- U9 pad 39: (no net) -> Net-(U9-Pad39)
- U9 pad 40: (no net) -> Net-(U9-Pad40)
- U9 pad 41: (no net) -> Net-(U9-Pad41)
- U9 pad 55: (no net) -> Net-(U9-Pad55)
- U9 pad 56: (no net) -> Net-(U9-Pad56)
- U9 pad 60: (no net) -> Net-(U9-Pad60)
- U9 pad 61: (no net) -> Net-(U9-Pad61)
- U9 pad 62: (no net) -> Net-(U9-Pad62)
- U9 pad 63: (no net) -> Net-(U9-Pad63)
- U9 pad 65: (no net) -> Net-(U9-Pad65)
- U9 pad 66: (no net) -> Net-(U9-Pad66)
- U9 pad 67: (no net) -> Net-(U9-Pad67)
- U9 pad 68: (no net) -> Net-(U9-Pad68)
- U9 pad 69: (no net) -> Net-(U9-Pad69)
- U9 pad 70: (no net) -> Net-(U9-Pad70)
- U9 pad 71: (no net) -> Net-(U9-Pad71)
- U9 pad 72: (no net) -> Net-(U9-Pad72)
- U9 pad 74: (no net) -> Net-(U9-Pad74)
- U9 pad 75: (no net) -> Net-(U9-Pad75)
- U9 pad 77: (no net) -> Net-(U9-Pad77)
- U9 pad 78: (no net) -> Net-(U9-Pad78)
- U9 pad 79: (no net) -> Net-(U9-Pad79)
- U9 pad 80: (no net) -> Net-(U9-Pad80)
- U9 pad 81: (no net) -> Net-(U9-Pad81)
- U9 pad 82: (no net) -> Net-(U9-Pad82)
- U9 pad 83: (no net) -> Net-(U9-Pad83)
- U9 pad 84: (no net) -> Net-(U9-Pad84)
- U9 pad 86: (no net) -> Net-(U9-Pad86)
- U9 pad 87: (no net) -> Net-(U9-Pad87)
- U9 pad 88: (no net) -> Net-(U9-Pad88)
- U9 pad 9: (no net) -> Net-(U9-Pad9)
- U9 pad 90: (no net) -> Net-(U9-Pad90)
- U9 pad 91: (no net) -> Net-(U9-Pad91)
- U9 pad 92: (no net) -> Net-(U9-Pad92)
- U9 pad 93: (no net) -> Net-(U9-Pad93)
- U9 pad 94: (no net) -> Net-(U9-Pad94)
- UARTCAN0 pad 9: (no net) -> Net-(UARTCAN0-Pad9)
- UARTCAN1 pad 9: (no net) -> Net-(UARTCAN1-Pad9)
- UARTCAN2 pad 9: (no net) -> Net-(UARTCAN2-Pad9)
- VR1 pad 4: (no net) -> Net-(VR1-Pad4)
Routing:
- net Net-(J1-Pad3): track 33.0 -> 31.0 mm

Commit message: New upstream version 5.0.0~rc2+dfsg1
Parts:
- ALLPST1, CLKOUT1, GND1, RS1, TA-1, VREF1: footprint connect:PINTST -> Connector_PinHeader_2.54mm:PinHeader_1x01_P2.54mm_Vertical
- BDM_EN1, CAN_TERM1, CLK0, CLK1, CT1, LED_EN1, VDDA1, VX_EN1: footprint pin_array:PIN_ARRAY_2X1 -> Connector_PinHeader_2.54mm:PinHeader_1x02_P2.54mm_Vertical
- BDM_PORT1: footprint pin_array:pin_array_13x2 -> Connector_PinHeader_2.54mm:PinHeader_2x13_P2.54mm_Vertical
- C1, C10, C11, C12, C14, C15, C18, C2, C20, C21, C22, C23, C24, C25, C26, C27, C28, C3, C30, C31, C32, C33, C34, C35, C36, C4, C41, C43, C44, C45, C46, C5, C51, C52, C53, C54, C55, C56, C57, C58, C59, C6, C60, C61, C7, C8, C9, R1, R10, R11, R12, R13, R14, R15, R16, R17, R18, R19, R2, R20, R22, R23, R25, R26, R28, R30, R31, R32, R33, R34, R35, R36, R38, R4, R45, R46, R47, R48, R49, R5, R50, R53, R57, R6, R62, R63, R7, R8, R9, RCAN1, RCAN2: footprint lib_smd:SM0805 -> Resistor_SMD:R_0805_2012Metric
- C38, C40: footprint discret:C2V8 -> Capacitor_THT:CP_Radial_D8.0mm_P5.00mm
- CAN_EN1, P3: footprint pin_array:PIN_ARRAY_2X2 -> Connector_PinHeader_2.54mm:PinHeader_2x02_P2.54mm_Vertical
- COM_SEL1, COM_SEL2, COM_SEL3: footprint pin_array:PIN_ARRAY_3X1 -> Connector_PinHeader_2.54mm:PinHeader_1x03_P2.54mm_Vertical
- D1, D3: footprint lib_smd:ST23AK#1 -> Diode_SMD:D_SOT-23_ANK
- D7: footprint discret:D5 -> Diode_THT:D_DO-15_P12.70mm_Horizontal
- D8, D9, LED1, LED2, LED3, LED4, LED5: footprint lib_smd:SM1206POL -> LED_SMD:LED_1206_3216Metric
- FB1, L1, L2: footprint lib_smd:SM1206 -> Resistor_SMD:R_1206_3216Metric_Pad1.24x1.80mm_HandSolder
- LV1: footprint discret:TO92-INVERT -> TO_SOT_Packages_THT:TO-92_Molded_Narrow
- MCU_PORT1: footprint pin_array:PIN_ARRAY_30X2 -> Connector_PinHeader_2.54mm:PinHeader_2x30_P2.54mm_Vertical
- P1: footprint pin_array:PIN_ARRAY-6X1 -> Connector_PinHeader_2.54mm:PinHeader_1x06_P2.54mm_Vertical
- P4: footprint pin_array:PIN_ARRAY_20X2 -> Connector_PinHeader_2.54mm:PinHeader_2x20_P2.54mm_Vertical
- PULUPEN1, UART_EN0, UART_EN1, UART_EN2: footprint pin_array:pin_array_4x2 -> Connector_PinHeader_2.54mm:PinHeader_2x04_P2.54mm_Vertical
- R21: value 4,7K -> 4.7K; footprint lib_smd:SM0805 -> Resistor_SMD:R_0805_2012Metric
- R64: footprint discret:R4 -> Resistor_THT:R_Axial_DIN0207_L6.3mm_D2.5mm_P10.16mm_Horizontal
- U1: footprint lib_smd:VQFP100 -> Package_QFP:LQFP-100_14x14mm_P0.5mm
- U3, U5, U8: footprint lib_smd:SO16E -> Package_SO:SOIC-16_3.9x9.9mm_P1.27mm
- U4: footprint lib_smd:SO14E -> Package_SO:SOIC-14_3.9x8.7mm_P1.27mm
- U7: footprint lib_smd:SO8E -> Package_SO:SOIC-8_3.9x4.9mm_P1.27mm
- U9: footprint lib_smd:TQFP144 -> Package_QFP:TQFP-144_20x20mm_P0.5mm
- VR1: footprint lib_smd:DPAK5 -> Package_TO_SOT_SMD:TO-263-5_TabPin3
- Y1: footprint discret:HC-18UH -> Crystal:Crystal_HC18-U_Horizontal
- moved MCU_PORT1 36.9 mm to (184.4, 136.9), turned to 270 degrees
- moved P4 24.2 mm to (222.2, 88.9), turned to 0 degrees
- moved BDM_PORT1 15.3 mm to (76.3, 106.3), turned to 0 degrees
- moved D7 6.35 mm to (93.5, 77.1), turned to 180 degrees
- moved P1 6.35 mm to (223.5, 63.5), turned to 0 degrees
- moved R64 5.08 mm to (207.0, 134.6)
- moved VR1 4.83 mm to (78.1, 88.3), turned to 90 degrees
- moved PULUPEN1 4.02 mm to (165.2, 118.0), turned to 270 degrees
- moved UART_EN1 4.02 mm to (169.5, 74.5), turned to 0 degrees
- moved UART_EN0 4.02 mm to (197.5, 74.5), turned to 0 degrees
- moved UART_EN2 4.02 mm to (135.8, 74.5), turned to 0 degrees
- moved COM_SEL1 2.54 mm to (113.3, 78.6), turned to 180 degrees
- moved COM_SEL2 2.54 mm to (110.7, 78.6), turned to 180 degrees
- moved COM_SEL3 2.54 mm to (108.2, 78.6), turned to 180 degrees
- moved C38 2.54 mm to (88.9, 87.6)
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Connections:
- net /inout_user/CANRX renamed /CANRX
- net /inout_user/CANTX renamed /CANTX
- net /inout_user/PWM1 renamed /PWM1
- net /inout_user/PWM3 renamed /PWM3
- net /inout_user/PWM5 renamed /PWM5
- net /inout_user/PWM7 renamed /PWM7
- net /inout_user/QSPI_DIN renamed /QSPI_DIN
- net /inout_user/QSPI_DOUT renamed /DSPI_DOUT
- net /inout_user/QSPI_SCLK renamed /QSPI_CLK
- net /inout_user/RCON- renamed /RCON-
- net /inout_user/RTS0- renamed /RSTO-
- net /inout_user/UCTS0 renamed /UCTS0
- net /inout_user/UCTS1 renamed /UCTS1
- net /inout_user/UCTS2 renamed /UCTS2
- net /inout_user/URTS0 renamed /URTS0
- net /inout_user/URTS1 renamed /URTS1
- net /inout_user/URTS2 renamed /URTS2
- net /inout_user/URXD0 renamed /URXD0
- net /inout_user/URXD1 renamed /URXD1
- net /inout_user/URXD2 renamed /URXD2
- net /inout_user/UTXD0 renamed /UTXD0
- net /inout_user/UTXD1 renamed /UTXD1
- net /inout_user/UTXD2 renamed /UTXD2
- net /inout_user/VCCA renamed /VCCA
- net /xilinx/GLCK2 renamed /XTAL
- net /xilinx/IRQ-1 renamed /IRQ-1
- net /xilinx/IRQ-2 renamed /IRQ-2
- net /xilinx/IRQ-3 renamed /IRQ-3
- net /xilinx/QSPI_CS1 renamed /QSPI_CS1
- net /xilinx/QSPI_CS2 renamed /QSPI_CS2
- BDM_PORT1 pad 1: Net-(BDM_PORT1-Pad1) -> (no net)
- BDM_PORT1 pad 21: Net-(BDM_PORT1-Pad21) -> (no net)
- BDM_PORT1 pad 22: Net-(BDM_PORT1-Pad22) -> (no net)
- BDM_PORT1 pad 7: /inout_user/RSTI- -> /RSTI-
- D1 pad 1: /IRQ-7 -> Net-(D1-Pad1)
- D1 pad 2: Net-(D1-Pad2) -> /IRQ-7
- D3 pad 1: /inout_user/RSTI- -> Net-(C3-Pad1)
- D3 pad 2: Net-(C3-Pad1) -> /RSTI-
- D7 pad 1: GND -> Net-(C38-Pad1)
- D7 pad 2: Net-(C38-Pad1) -> GND
- MCU_PORT1 pad 6: /inout_user/RSTI- -> /RSTI-
- R14 pad 2: Net-(D1-Pad2) -> Net-(D1-Pad1)
- R15 pad 2: /inout_user/RSTI- -> /RSTI-
- SW_ONOFF1 pad 1: Net-(SW_ONOFF1-Pad1) -> (no net)
- U1 pad 96: /inout_user/RSTI- -> /RSTI-
- U2 pad 4: Net-(D1-Pad2) -> Net-(D1-Pad1)
- U9 pad 102: Net-(U9-Pad102) -> (no net)
- U9 pad 103: Net-(U9-Pad103) -> (no net)
- U9 pad 106: Net-(U9-Pad106) -> (no net)
- U9 pad 110: Net-(U9-Pad110) -> (no net)
- U9 pad 120: Net-(U9-Pad120) -> (no net)
- U9 pad 121: Net-(U9-Pad121) -> (no net)
- U9 pad 133: Net-(U9-Pad133) -> (no net)
- U9 pad 14: Net-(U9-Pad14) -> (no net)
- U9 pad 141: Net-(U9-Pad141) -> (no net)
- U9 pad 15: Net-(U9-Pad15) -> (no net)
- U9 pad 16: Net-(U9-Pad16) -> (no net)
- U9 pad 18: Net-(U9-Pad18) -> (no net)
- U9 pad 19: Net-(U9-Pad19) -> (no net)
- U9 pad 21: Net-(U9-Pad21) -> (no net)
- U9 pad 22: Net-(U9-Pad22) -> (no net)
- U9 pad 23: Net-(U9-Pad23) -> (no net)
- U9 pad 25: Net-(U9-Pad25) -> (no net)
- U9 pad 26: Net-(U9-Pad26) -> (no net)
- U9 pad 29: Net-(U9-Pad29) -> (no net)
- U9 pad 30: Net-(U9-Pad30) -> (no net)
- U9 pad 34: Net-(U9-Pad34) -> (no net)
- U9 pad 35: Net-(U9-Pad35) -> (no net)
- U9 pad 36: Net-(U9-Pad36) -> (no net)
- U9 pad 37: Net-(U9-Pad37) -> (no net)
- U9 pad 38: Net-(U9-Pad38) -> (no net)
- U9 pad 39: Net-(U9-Pad39) -> (no net)
- U9 pad 40: Net-(U9-Pad40) -> (no net)
- U9 pad 41: Net-(U9-Pad41) -> (no net)
- U9 pad 55: Net-(U9-Pad55) -> (no net)
- U9 pad 56: Net-(U9-Pad56) -> (no net)
- U9 pad 60: Net-(U9-Pad60) -> (no net)
- U9 pad 61: Net-(U9-Pad61) -> (no net)
- U9 pad 62: Net-(U9-Pad62) -> (no net)
- U9 pad 63: Net-(U9-Pad63) -> (no net)
- U9 pad 65: Net-(U9-Pad65) -> (no net)
- U9 pad 66: Net-(U9-Pad66) -> (no net)
- U9 pad 67: Net-(U9-Pad67) -> (no net)
- U9 pad 68: Net-(U9-Pad68) -> (no net)
- U9 pad 69: Net-(U9-Pad69) -> (no net)
- U9 pad 70: Net-(U9-Pad70) -> (no net)
- U9 pad 71: Net-(U9-Pad71) -> (no net)
- U9 pad 72: Net-(U9-Pad72) -> (no net)
- U9 pad 74: Net-(U9-Pad74) -> (no net)
- U9 pad 75: Net-(U9-Pad75) -> (no net)
- U9 pad 77: Net-(U9-Pad77) -> (no net)
- U9 pad 78: Net-(U9-Pad78) -> (no net)
- U9 pad 79: Net-(U9-Pad79) -> (no net)
- U9 pad 80: Net-(U9-Pad80) -> (no net)
- U9 pad 81: Net-(U9-Pad81) -> (no net)
- U9 pad 82: Net-(U9-Pad82) -> (no net)
- U9 pad 83: Net-(U9-Pad83) -> (no net)
- U9 pad 84: Net-(U9-Pad84) -> (no net)
- U9 pad 86: Net-(U9-Pad86) -> (no net)
- U9 pad 87: Net-(U9-Pad87) -> (no net)
- U9 pad 88: Net-(U9-Pad88) -> (no net)
- U9 pad 9: Net-(U9-Pad9) -> (no net)
- U9 pad 90: Net-(U9-Pad90) -> (no net)
- U9 pad 91: Net-(U9-Pad91) -> (no net)
- U9 pad 92: Net-(U9-Pad92) -> (no net)
- U9 pad 93: Net-(U9-Pad93) -> (no net)
- U9 pad 94: Net-(U9-Pad94) -> (no net)
- UARTCAN0 pad 9: Net-(UARTCAN0-Pad9) -> (no net)
- UARTCAN1 pad 9: Net-(UARTCAN1-Pad9) -> (no net)
- UARTCAN2 pad 9: Net-(UARTCAN2-Pad9) -> (no net)
- VR1 pad 4: Net-(VR1-Pad4) -> (no net)
Routing:
- net /inout_user/RSTI-: track 207.4 -> 0.00 mm, vias 2 -> 0
- net /RSTI-: track 0.00 -> 207.4 mm, vias 0 -> 2
- net Net-(D1-Pad2): track 10.9 -> 0.00 mm
- net Net-(D1-Pad1): track 0.00 -> 10.9 mm
- net +3.3V: track 983.5 -> 994.3 mm
- net Net-(C38-Pad1): track 41.5 -> 45.5 mm
- net GND: track 1134.9 -> 1137.8 mm
- net /xilinx/TDI: track 42.5 -> 44.9 mm
- net Net-(L1-Pad1): track 2.44 -> 4.45 mm
- net /inout_user/RxD_CAN: track 6.77 -> 8.51 mm
- net /xilinx/TMS: track 43.3 -> 44.7 mm
- net /xilinx/TCK: track 66.1 -> 67.5 mm
- net /xilinx/XIL_D20: track 25.8 -> 27.1 mm
- net /inout_user/CAN_H: track 27.5 -> 28.7 mm
- net Net-(F1-Pad1): track 15.4 -> 14.4 mm
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