File: demos/sonde xilinx/sonde xilinx.kicad_pcb (KiCad board)
At the start: 2 copper layers, 29 parts, among them J1 DB25MALE, J2 DB9MALE, P1 CONN_6, U1 74LS125, U2 74LS125

Commit message: Imported Upstream version 4.0.0~rc1
Parts:
- removed MIRE (x4): *, MIRE
Other:
- board outline added: 81.3 x 43.2 mm
