File: demos/test_xil_95108/carte_test.kicad_pcb (KiCad board)
At the start: 2 copper layers, 42 parts, among them J1 DB25, J2 DB9FEM, K1 CONN_3, P2 CONN_3, P3 CONN_2, P4 CONN_2X2, SW1 SW_PUSH, SW2 SW_PUSH, U1 TDA8702, U2 XC95108PC84, U3 LM7805, U4 74HC04, U5 RAM_32KO, U6 LM318N, X1 10MHz

Commit message: Imported Upstream version 4.0.0~rc1
Connections:
- net CSMEM_1 renamed /CSMEM
- net DAT0_1 renamed /DAT0
- net DAT1_1 renamed /DAT1
- net DAT2_1 renamed /DAT2
- net DAT3_1 renamed /DAT3
- net DAT4_1 renamed /DAT4
- net DAT5_1 renamed /DAT5
- net DAT6_1 renamed /DAT6
- net DAT7_1 renamed /DAT7
- net DCLK_1 renamed /DCLK
- net LED1_1 renamed /LED1
- net LED2_1 renamed /LED2
- net MA0_1 renamed /MA0
- net MA1_1 renamed /MA1
- net MA2_1 renamed /MA2
- net MA3_1 renamed /MA3
- net MA4_1 renamed /MA4
- net MA5_1 renamed /MA5
- net MA6_1 renamed /MA6
- net MA7_1 renamed /MA7
- net MD0_1 renamed /MD0
- net MD10_1 renamed /MD10
- net MD11_1 renamed /MD11
- net MD12_1 renamed /MD12
- net MD13_1 renamed /MD13
- net MD14_1 renamed /MD14
- net MD1_1 renamed /MD1
- net MD2_1 renamed /MD2
- net MD3_1 renamed /MD3
- net MD4_1 renamed /MD4
- net MD5_1 renamed /MD5
- net MD6_1 renamed /MD6
- net MD7_1 renamed /MD7
- net MD8_1 renamed /MD8
- net MD9_1 renamed /MD9
- net OEMEM_1 renamed /OEMEM
- net PARBUS0_1 renamed /PARBUS0
- net PARBUS1_1 renamed /PARBUS1
- net PARBUS2_1 renamed /PARBUS2
- net PARBUS3_1 renamed /PARBUS3
- net PARBUS4_1 renamed /PARBUS4
- net PARBUS5_1 renamed /PARBUS5
- net PARBUS6_1 renamed /PARBUS6
- net PARBUS7_1 renamed /PARBUS7
- net PAR_AUX0_X00001 renamed /PAR_AUX0/STROBE*
- net PAR_AUX1_X00004 renamed /PAR_AUX1/ERROR*
- net PAR_AUX2_X00003 renamed /PAR_AUX2/AUTOLF*
- net PAR_AUX3_X00002 renamed /PAR_AUX3/SELECT*
- net PAR_AUX4/PE_1 renamed /PAR_AUX4/PE
- net PAR_AUX5/BUSY*_1 renamed /PAR_AUX5/BUSY*
- net PAR_AUX6/ACK_1 renamed /PAR_AUX6/ACK
- net PAR_AUX7/INIT_1 renamed /PAR_AUX7/INIT
- net PAR_AUX8_X00005 renamed /PAR_AUX8/SELECT
- net PIN_TEST0_1 renamed /PIN_TEST0
- net PIN_TEST1_1 renamed /PIN_TEST1
- net R/W-A14_1 renamed /R/W-A14
- net SW0_1 renamed /SW0
- net SW1_1 renamed /SW1
- net TCK_1 renamed /TCK
- net TDI_1 renamed /TDI
- net TDO_1 renamed /TDO
- net TMS_1 renamed /TMS
- net XIN/CLK_1 renamed /XIN/CLK
Other:
- board outline added: 101.6 x 99.7 mm
