File: demos/test_xil_95108/carte_test.kicad_pcb (KiCad board)
At the start: 2 copper layers, 101.6 x 99.7 mm, 42 parts, among them J1 DB25, J2 DB9FEM, K1 CONN_3, P2 CONN_3, P3 CONN_2, P4 CONN_2X2, SW1 SW_PUSH, SW2 SW_PUSH, U1 TDA8702, U2 XC95108PC84, U3 LM7805, U4 74HC04, U5 RAM_32KO, U6 LM318N, X1 10MHz

Commit message: New upstream version 5.0.0~rc1+dfsg1
Parts:
- C10, C11, C7, C8: footprint Capacitors_SMD:C_1206 -> Capacitor_SMD:C_1206_3216Metric_Pad1.24x1.80mm_HandSolder
- C13, C14, C2, C3, C6: footprint Discret:CP6 -> Capacitor_THT:CP_Axial_L10.0mm_D4.5mm_P15.00mm_Horizontal
- D2, D3: footprint LEDs:LED-5MM -> LED_THT:LED_D5.0mm
- J1: footprint Connect:DB25FC -> Connector_Dsub:DSUB-25_Female_Horizontal_P2.77x2.84mm_EdgePinOffset9.90mm_Housed_MountingHolesOffset11.32mm
- J2: footprint Connect:DB9F_CI_INVERT -> Connector_Dsub:DSUB-9_Female_EdgeMount_P2.77mm; moved to B.Cu
- P2: footprint Socket_Strips:Socket_Strip_Straight_1x03 -> TerminalBlock_Phoenix:TerminalBlock_Phoenix_MKDS-1,5-3-5.08_1x03_P5.08mm_Horizontal
- P3: footprint Connect:bornier2 -> TerminalBlock_Phoenix:TerminalBlock_Phoenix_MKDS-1,5-2-5.08_1x02_P5.08mm_Horizontal
- R1, R10, R2, R3, R4, R5, R6, R7, R8, R9: footprint Discret:R4 -> Resistor_THT:R_Axial_DIN0207_L6.3mm_D2.5mm_P10.16mm_Horizontal
- U1: footprint Sockets_DIP:DIP-16__300_ELL -> Package_DIP:DIP-16_W7.62mm_Socket_LongPads
- U3: footprint Discret:LM78XX -> TO_SOT_Packages_THT:TO-220_Horizontal
- U6: footprint Sockets_DIP:DIP-8__300_ELL -> Package_DIP:DIP-8_W7.62mm_LongPads
- X1: footprint Crystals:HC-18UH -> Crystal:Crystal_HC18-U_Horizontal
- moved J1 16.7 mm to (102.2, 104.9), turned to 270 degrees
- moved D1 10.7 mm to (181.1, 121.9), turned to 90 degrees
- moved U1 9.67 mm to (123.8, 65.4), turned to 90 degrees
- moved C6 7.92 mm to (164.0, 108.3)
- moved C13 7.62 mm to (167.0, 43.9)
- moved C14 7.62 mm to (129.5, 50.2)
- moved C2 7.62 mm to (129.5, 54.0)
- moved C3 7.62 mm to (188.6, 81.3)
- moved P2 5.97 mm to (189.7, 130.6)
- moved U6 5.39 mm to (121.9, 47.0), turned to 90 degrees
- moved R7 5.38 mm to (134.6, 40.1)
- moved R8 5.16 mm to (134.6, 43.6)
- moved R1 5.08 mm to (125.1, 126.4)
- moved R4 5.08 mm to (150.5, 64.1)
- moved R5 5.08 mm to (148.0, 64.1)
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Routing:
- net GND: track 361.0 -> 314.1 mm
- net +12V: track 168.7 -> 179.1 mm
- net /-12BATT: track 26.6 -> 17.4 mm
- net Net-(P3-Pad1): track 6.98 -> 15.1 mm
- net /SW0: track 62.8 -> 58.0 mm
- net /SW1: track 75.5 -> 70.9 mm
- net /+12BATT: track 14.2 -> 10.3 mm
- net /TDO: track 154.6 -> 157.8 mm
- net -12V: track 118.9 -> 120.1 mm
- net VCC: track 345.6 -> 344.5 mm
- net Net-(R10-Pad2): track 64.1 -> 64.9 mm
- net /MA3: track 68.1 -> 69.0 mm
- net Net-(C14-Pad2): track 8.78 -> 9.60 mm
- net /MA4: track 60.7 -> 61.4 mm
