File: demos/test_xil_95108/carte_test.sch (KiCad schematic (older format))
At the start: 42 parts, among them J1 DB25, J2 DB9FEM, K1 CONN_3, P2 CONN_3, P3 CONN_2, P4 CONN_2X2, SW1 SW_PUSH, SW2 SW_PUSH, U1 TDA8702, U2 XC95108PC84, U3 LM7805, U4 74HC04, U5 RAM_32KO, U6 LM318N, X1 10MHz

Commit message: Imported Upstream version 4.0.0~rc1
Connections:
- wire segments 191 -> 251
Other:
- moved on the sheet: U3, U4B
