File: demos/test_xil_95108/carte_test.sch (KiCad schematic (older format))
At the start: 42 parts, among them J1 DB25, J2 DB9FEM, K1 CONN_3, P2 CONN_3, P3 CONN_2, P4 CONN_2X2, SW1 SW_PUSH, SW2 SW_PUSH, U1 TDA8702, U2 XC95108PC84, U3 LM7805, U4 74HC04, U5 RAM_32KO, U6 LM318N, X1 10MHz

Commit message: New upstream version 5.0.0~rc1+dfsg1
Parts:
- C1, C12, C4, C5: symbol C -> carte_test_schlib:C
- C10, C11, C7, C8: footprint Capacitors_SMD:C_1206 -> Capacitor_SMD:C_1206_3216Metric_Pad1.24x1.80mm_HandSolder; symbol C -> carte_test_schlib:C
- C13, C14, C2, C3, C6: footprint Discret:CP6 -> Capacitor_THT:CP_Axial_L10.0mm_D4.5mm_P15.00mm_Horizontal; symbol CP -> carte_test_schlib:CP
- D1, D4: symbol DIODE -> carte_test_schlib:DIODE
- D2, D3: footprint LEDs:LED-5MM -> LED_THT:LED_D5.0mm; symbol LED -> carte_test_schlib:LED
- J1: footprint Connect:DB25FC -> Connector_Dsub:DSUB-25_Female_Horizontal_P2.77x2.84mm_EdgePinOffset9.90mm_Housed_MountingHolesOffset11.32mm; symbol DB25 -> carte_test_schlib:DB25
- J2: footprint Connect:DB9F_CI_INVERT -> Connector_Dsub:DSUB-9_Female_EdgeMount_P2.77mm; symbol DB9 -> carte_test_schlib:DB9
- K1: symbol CONN_3 -> carte_test_schlib:CONN_3
- P2: footprint Socket_Strips:Socket_Strip_Straight_1x03 -> TerminalBlock_Phoenix:TerminalBlock_Phoenix_MKDS-1,5-3-5.08_1x03_P5.08mm_Horizontal; symbol CONN_3 -> carte_test_schlib:CONN_3
- P3: footprint Connect:bornier2 -> TerminalBlock_Phoenix:TerminalBlock_Phoenix_MKDS-1,5-2-5.08_1x02_P5.08mm_Horizontal; symbol CONN_2 -> carte_test_schlib:CONN_2
- P4: symbol CONN_2X2 -> carte_test_schlib:CONN_2X2
- R1, R10, R2, R3, R4, R5, R6, R7, R8, R9: footprint Discret:R4 -> Resistor_THT:R_Axial_DIN0207_L6.3mm_D2.5mm_P10.16mm_Horizontal; symbol R -> carte_test_schlib:R
- SW1, SW2: symbol SW_PUSH -> carte_test_schlib:SW_PUSH
- U1: footprint Sockets_DIP:DIP-16__300_ELL -> Package_DIP:DIP-16_W7.62mm_Socket_LongPads; symbol TDA8702 -> carte_test_schlib:TDA8702
- U2: symbol XC95108PC84 -> carte_test_schlib:XC95108PC84
- U3: footprint Discret:LM78XX -> TO_SOT_Packages_THT:TO-220_Horizontal; symbol LM7805 -> carte_test_schlib:LM7805
- U4: symbol 74HC04 -> carte_test_schlib:74HC04
- U5: symbol RAM_32KO -> carte_test_schlib:RAM_32KO
- U6: footprint Sockets_DIP:DIP-8__300_ELL -> Package_DIP:DIP-8_W7.62mm_LongPads; symbol LM318N -> carte_test_schlib:LM318N
- X1: footprint Crystals:HC-18UH -> Crystal:Crystal_HC18-U_Horizontal; symbol CRYSTAL -> carte_test_schlib:CRYSTAL
Connections:
- wire segments 209 -> 241
