File: demos/electric/electric.sch (KiCad schematic (older format))
At the start: 97 parts

Commit message: Imported Upstream version 4.0.0~rc1
Parts:
- EC11, EC12, EC13, EC14, EC15, EC16, EC17, EC18, EC19, EC31, EC41, EC42, EC43, EC44: value C_3X1.5MM2 -> C_3x1.5mm2; symbol C_3X1.5MM2 -> C_3x1.5mm2
- EC20, EC21, EC22, EC23, EC24, EC25, EC26, EC28, EC29, EC30, EC32, EC33, EC34, EC35, EC36, EC37, EC38, EC39, EC? (x2): value C_3X2.5MM2 -> C_3x2.5mm2; symbol C_3X2.5MM2 -> C_3x2.5mm2
- EC27: value C_3X6MM2 -> C_3x6mm2; symbol C_3X6MM2 -> C_3x6mm2
- EG1: value G_TH_3KVA -> G_Th_3KVA; symbol G_TH_3KVA -> G_Th_3KVA; Champ4 (none) -> automatique; Champ5 (none) -> diesel
- EJ1, EJ2, EJ3, EJ4: value J_40A_30MA -> J_40A_30mA; symbol J_40A_30MA -> J_40A_30mA
- EO1: Champ4 (none) -> rallongée
- ER01, ER02: value R_16A_30MA -> R_16A_30mA; symbol R_16A_30MA -> R_16A_30mA
- EV2: symbol V_F50HZ -> V_F50Hz
Connections:
- wire segments 135 -> 82
Other:
- note added: "Servitudes\npermanentes\nprimaires"
- note added: "Servitudes\npermanentes\nsecondaires"
- note removed: "Servitudes"
- note removed: "permanentes"
- note removed: "primaires"
- note removed: "secondaires"

Commit message: New upstream version 5.0.0~rc1+dfsg1
Parts:
- removed ED11: D_06A, Eclairage vide sanitaire, symbol D_06A
- removed ED12: D_06A, Eclairage chambre 1, chambre 2, symbol D_06A
- removed ED13: D_06A, Eclairage séjour, cuisine, symbol D_06A
- removed ED14: D_06A, Eclairage chambre 3, couloir 2, symbol D_06A
- removed ED15: D_06A, Eclairage grange, symbol D_06A
- removed ED16: D_06A, Informatique, symbol D_06A
- removed ED20: D_10A, Vide sanitaire, portail, symbol D_10A
- removed ED21: D_10A, Pompe surpresseur, symbol D_10A
- removed ED22: D_10A, Réfrigérateur & congélateur, symbol D_10A
- removed ED25: D_10A, Matériel sensible, symbol D_10A
- removed ED31: D_06A, Chauffage, symbol D_06A
- removed ED32: D_06A, Traitement de l'eau, symbol D_06A
- removed ED33: D_06A, Silveloxs, volets, symbol D_06A
- removed ED50: D_16A, Chambre 1, symbol D_16A
- removed ED51: D_16A, Chambre 2, symbol D_16A
- removed ED52: D_16A, Chambre 3, symbol D_16A
- removed ED53: D_16A, Bureau, symbol D_16A
- removed ED54: D_16A, Séjour et sam, symbol D_16A
- removed ED60: D_16A, Atelier, symbol D_16A
- removed ED61: D_16A, Sellerie, symbol D_16A
- removed ED62: D_16A, Local technique, symbol D_16A
- removed ED63: D_16A, Etage coté sellerie, symbol D_16A
- removed ED64: D_16A, Etage coté atelier, symbol D_16A
- removed ED70: D_10A, Abri coté route, symbol D_10A
- removed ED71: D_10A, Abri pré Mouillière proche, symbol D_10A
- removed ED72, ED73: D_10A, symbol D_10A
- added ED11: D_06A, Eclairage vide sanitaire, symbol elec-unifil:D_06A
- added ED12: D_06A, Eclairage chambre 1, chambre 2, symbol elec-unifil:D_06A
- added ED13: D_06A, Eclairage séjour, cuisine, symbol elec-unifil:D_06A
- added ED14: D_06A, Eclairage chambre 3, couloir 2, symbol elec-unifil:D_06A
- added ED15: D_06A, Eclairage grange, symbol elec-unifil:D_06A
- added ED16: D_06A, Informatique, symbol elec-unifil:D_06A
- added ED20: D_10A, Vide sanitaire, portail, symbol elec-unifil:D_10A
- added ED21: D_10A, Pompe surpresseur, symbol elec-unifil:D_10A
- added ED22: D_10A, Réfrigérateur & congélateur, symbol elec-unifil:D_10A
- added ED25: D_10A, Matériel sensible, symbol elec-unifil:D_10A
- added ED31: D_06A, Chauffage, symbol elec-unifil:D_06A
- added ED32: D_06A, Traitement de l'eau, symbol elec-unifil:D_06A
- added ED33: D_06A, Silveloxs, volets, symbol elec-unifil:D_06A
- added ED50: D_16A, Chambre 1, symbol elec-unifil:D_16A
- added ED51: D_16A, Chambre 2, symbol elec-unifil:D_16A
- added ED52: D_16A, Chambre 3, symbol elec-unifil:D_16A
- added ED53: D_16A, Bureau, symbol elec-unifil:D_16A
- added ED54: D_16A, Séjour et sam, symbol elec-unifil:D_16A
- added ED60: D_16A, Atelier, symbol elec-unifil:D_16A
- added ED61: D_16A, Sellerie, symbol elec-unifil:D_16A
- added ED62: D_16A, Local technique, symbol elec-unifil:D_16A
- added ED63: D_16A, Etage coté sellerie, symbol elec-unifil:D_16A
- added ED64: D_16A, Etage coté atelier, symbol elec-unifil:D_16A
- added ED70: D_10A, Abri coté route, symbol elec-unifil:D_10A
- added ED71: D_10A, Abri pré Mouillière proche, symbol elec-unifil:D_10A
- added ED72, ED73: D_10A, symbol elec-unifil:D_10A
- EA1: symbol A_1KVA -> elec-unifil:A_1KVA
- EC101, EC102: renamed from EC?; symbol C_3x2.5mm2 -> elec-unifil:C_3x2.5mm2
- EC11, EC12, EC13, EC14, EC15, EC16, EC17, EC18, EC19, EC31, EC41, EC42, EC43, EC44: symbol C_3x1.5mm2 -> elec-unifil:C_3x1.5mm2
- EC20, EC21, EC22, EC23, EC24, EC25, EC26, EC28, EC29, EC30, EC32, EC33, EC34, EC35, EC36, EC37, EC38, EC39: symbol C_3x2.5mm2 -> elec-unifil:C_3x2.5mm2
- EC27: symbol C_3x6mm2 -> elec-unifil:C_3x6mm2
- ED10, ED43, ED44, ED47: symbol D_10A -> elec-unifil:D_10A
- ED30: symbol D_06A -> elec-unifil:D_06A
- ED40: symbol D_32A -> elec-unifil:D_32A
- ED41, ED42, ED45, ED46, ED55: symbol D_16A -> elec-unifil:D_16A
- EG1: symbol G_Th_3KVA -> elec-unifil:G_Th_3KVA
- EI11: symbol I_25A_LUM -> elec-unifil:I_25A_LUM
- EJ1, EJ2, EJ3, EJ4: symbol J_40A_30mA -> elec-unifil:J_40A_30mA
- EO1: symbol O_900VA -> elec-unifil:O_900VA
- EO2: symbol O_600VA -> elec-unifil:O_600VA
- EP4: symbol P_10A -> elec-unifil:P_10A
- EQ1a101: renamed from EQ1a; symbol Q_25A_2F2O -> elec-unifil:Q_25A_2F2O
- EQ1b101: renamed from EQ1b; symbol Q_25A_2F2O -> elec-unifil:Q_25A_2F2O
- EQ2, EQ3: symbol Q_25A_2F2O -> elec-unifil:Q_25A_2F2O
- EQ4: symbol Q_2A_12O_40KV -> elec-unifil:Q_2A_12O_40KV
- ER1: renamed from ER01; symbol R_16A_30mA -> elec-unifil:R_16A_30mA
- ER2: renamed from ER02; symbol R_16A_30mA -> elec-unifil:R_16A_30mA
- ES1: symbol S_63A -> elec-unifil:S_63A
- EV1: symbol V_A10A -> elec-unifil:V_A10A
- EV2: symbol V_F50Hz -> elec-unifil:V_F50Hz
- EV3: symbol V_U400V -> elec-unifil:V_U400V
- EW1: renamed from EW01; symbol W_15KA -> elec-unifil:W_15KA
- EY1, EY2: symbol Y_ELC -> elec-unifil:Y_ELC
Connections:
- net at EJ2.1: now also ED60.2, ED61.2, ED62.2, ED63.2, ED64.2
- net at ED55.2, EJ3.1: now also ED50.2, ED51.2, ED52.2, ED53.2, ED54.2
- net at EJ4.1: now also ED70.2, ED71.2, ED72.2, ED73.2
- net at EV3.1: now also ED20.2, ED21.2, ED22.2
- net at EQ4.24: now also ED25.2
- net at EO1.1: now also ED11.2, ED12.2, ED13.2, ED14.2, ED15.2, ED16.2
- net at ED30.2, EO2.1: now also ED31.2, ED32.2, ED33.2
- net at EC12.2: now also ED20.1
- net at EC11.2: now also ED11.1
- net at EC41.2: now also ED31.1
- net at EC17.2: now also ED21.1
- net at EC31.2: now also ED22.1
- net at EC18.2: now also ED25.1
- net at EC13.2: now also ED12.1
- net at EC14.2: now also ED13.1
- net at EC15.2: now also ED14.1
- net at EC16.2: now also ED15.1
- net at EC42.2: now also ED16.1
- net at EC43.2: now also ED32.1
- net at EC44.2: now also ED33.1
- net at EC34.2: now also ED60.1
- net at EC36.2: now also ED61.1
- net at EC35.2, EP4.1: now also ED62.1
- net at EC38.2: now also ED63.1
- net at EC39.2: now also ED64.1
- net at EC20.2: now also ED50.1
- net at EC21.2: now also ED51.1
- net at EC33.2: now also ED52.1
- net at EC37.2: now also ED53.1
- net at EC22.2: now also ED54.1
- net at EC101.2: now also ED70.1
- net at EC102.2: now also ED71.1
Other:
- moved on the sheet: ED13, ED14, ED60, ED64
