File: demos/pspice/pspice.sch (KiCad schematic (older format))
At the start: 20 parts, among them Q1 Q2N2222, Q2 Q2N2222, Q3 Q2N2222

Commit message: Imported Upstream version 4.0.0~rc1
Connections:
- wire segments 23 -> 40
Other:
- moved on the sheet: C3, L1, R10, R11, R7, R8

Commit message: New upstream version 5.0.0~rc1+dfsg1
Parts:
- removed R10: 220, symbol R
- added C4: 10nF, symbol schematic_libspice:CAP
- added L2: 100mH, symbol schematic_libspice:INDUCTOR
- added R12: 100, symbol schematic_libspice:R
- added R7: 22K, symbol schematic_libspice:R
- C1: symbol C -> schematic_libspice:C
- C2: value 1nF -> 220pF; symbol C -> schematic_libspice:C
- C3: value 10uF -> 10nF; symbol CAP -> schematic_libspice:CAP
- L1: symbol INDUCTOR -> schematic_libspice:INDUCTOR
- Q1: renamed from Q3; symbol QNPN -> schematic_libspice:QNPN
- Q2: renamed from Q1; symbol QNPN -> schematic_libspice:QNPN
- Q3: renamed from Q2; symbol QNPN -> schematic_libspice:QNPN
- R1: renamed from R11; value 100 -> 10; symbol R -> schematic_libspice:R
- R10: renamed from R7; symbol R -> schematic_libspice:R
- R11: renamed from R1; symbol R -> schematic_libspice:R
- R2: renamed from R12; symbol R -> schematic_libspice:R
- R3: renamed from R6; symbol R -> schematic_libspice:R
- R4: renamed from R3; symbol R -> schematic_libspice:R
- R5: renamed from R4; symbol R -> schematic_libspice:R
- R6: renamed from R5; symbol R -> schematic_libspice:R
- R8: symbol R -> schematic_libspice:R
- R9: renamed from R2; symbol R -> schematic_libspice:R
- V1: value DC 12V -> DC 12; symbol VSOURCE -> schematic_libspice:VSOURCE
- V2: value AC 0.1 -> AC; symbol VSOURCE -> schematic_libspice:VSOURCE; Spice_Model (none) -> dc 0 ac 1; Spice_Netlist_Enabled (none) -> Y; Spice_Primitive (none) -> V
Connections:
- net labels added: VBASE
- wire segments 40 -> 50
Other:
- note added: ".model Q2N2222 npn (bf=200)\n.ac dec 100 10 1Meg\n"
- note removed: "+gnucap .model Q2N2222 npn (bf=200)\n.print tran v(nodes)\n.print dc v(nodes)\n.tran 10 10000 10 > pspice.dat\n"
- moved on the sheet: C3
